File: hx711/hx711.kicad_sch (KiCad schematic)
At the start: 8 parts, among them J1 Screw_Terminal_01x04, J2 Screw_Terminal_01x04, Q1 S8550, SW1 Rate Selector, U1 HX711

Commit message: made changes to the HX711 footprints and finihsed the pcb
Parts:
- Q1: footprint Package_TO_SOT_THT:TO-92_Inline -> Package_TO_SOT_SMD:TSOT-23
- SW1: footprint Button_Switch_SMD:SW_SPDT_CK-JS102011SAQN -> Button_Switch_SMD:SW_SPDT_PCM12
Changed lines of the file:
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@@
       (effects (font (size 1.27 1.27)))
     )
-    (property "Footprint" "Button_Switch_SMD:SW_SPDT_CK-JS102011SAQN" (at 139.7 101.6 0)
+    (property "Footprint" "Button_Switch_SMD:SW_SPDT_PCM12" (at 139.7 101.6 0)
       (effects (font (size 1.27 1.27)) hide)
     )
@@
       (effects (font (size 1.27 1.27)))
     )
-    (property "Footprint" "Package_TO_SOT_THT:TO-92_Inline" (at 107.315 58.42 0)
+    (property "Footprint" "Package_TO_SOT_SMD:TSOT-23" (at 107.315 58.42 0)
       (effects (font (size 1.27 1.27) italic) (justify left) hide)
     )
