File: hx711/hx711.kicad_sch (KiCad schematic)
At the start: 8 parts, among them J1 Screw_Terminal_01x04, J2 Screw_Terminal_01x04, Q1 S8550, SW1 Rate Selector, U1 HX711

Commit message: Removed resistor at the ina- termina
Parts:
- added C2: C, Capacitor_SMD:C_0402_1005Metric, symbol Device:C
- added R3: R, Resistor_SMD:R_0402_1005Metric, symbol Device:R
Connections:
- net GND: now also C2.2
- net at U1.6 (VBG): now also C2.1
- net at J1.2 (Pin_2): now also R3.1; no longer U1.8 (INA+)
- new net: R3.2, U1.8 (INA+)
- no-connect marks 4 -> 3
Other:
- note added: "2.7 - 5.5 V"
Changed lines of the file:
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@@
   (no_connect (at 101.6 101.6))
   (no_connect (at 101.6 99.06))
-  (no_connect (at 101.6 106.68))
-  (wire (pts (xy 101.6 91.44) (xy 86.36 91.44))
-    (stroke (width 0) (type default))
-  )
   (wire (pts (xy 116.84 60.96) (xy 116.84 71.12))
     (stroke (width 0) (type default))
@@
     (stroke (width 0) (type default))
   )
+  (wire (pts (xy 86.36 93.98) (xy 101.6 93.98))
+    (stroke (width 0) (type default))
+  )
   (wire (pts (xy 91.44 60.96) (xy 96.52 60.96))
     (stroke (width 0) (type default))
@@
     (stroke (width 0) (type default))
   )
+  (wire (pts (xy 86.36 91.44) (xy 90.805 91.44))
+    (stroke (width 0) (type default))
+  )
   (wire (pts (xy 100.33 48.26) (xy 101.6 48.26))
     (stroke (width 0) (type default))
@@
     (stroke (width 0) (type default))
   )
-  (wire (pts (xy 101.6 93.98) (xy 86.36 93.98))
-    (stroke (width 0) (type default))
-  )
   (wire (pts (xy 87.63 60.96) (xy 91.44 60.96))
     (stroke (width 0) (type default))
   )
+  (wire (pts (xy 98.425 91.44) (xy 101.6 91.44))
+    (stroke (width 0) (type default))
+  )
   (wire (pts (xy 116.84 60.96) (xy 123.19 60.96))
     (stroke (width 0) (type default))
@@
   (wire (pts (xy 101.6 81.28) (xy 91.44 81.28))
     (stroke (width 0) (type default))
+  )
+  (text "2.7 - 5.5 V" (at 132.08 65.405 0)
+    (effects (font (size 1.27 1.27)) (justify left bottom))
   )
   (label "AVDD" (at 96.52 81.28 0) (fields_autoplaced)
@@
         (path "/80bd3c70-df1b-4e0c-ae87-ddc7b6d2e4eb"
           (reference "#FLG01") (unit 1)
+        )
+      )
+    )
+  )
+  (symbol (lib_id "Device:R") (at 94.615 91.44 90) (unit 1)
+    (in_bom yes) (on_board yes) (dnp no)
+    (property "Reference" "R3" (at 94.615 88.9 90)
+      (effects (font (size 1.27 1.27)))
+    )
+    (property "Value" "R" (at 94.615 91.44 90)
+      (effects (font (size 1.27 1.27)))
+    )
+    (property "Footprint" "Resistor_SMD:R_0402_1005Metric" (at 94.615 93.218 90)
+      (effects (font (size 1.27 1.27)) hide)
+    )
+    (property "Datasheet" "~" (at 94.615 91.44 0)
+      (effects (font (size 1.27 1.27)) hide)
+    )
+    (pin "1")
+    (pin "2")
+    (instances
+      (project "hx711"
+        (path "/80bd3c70-df1b-4e0c-ae87-ddc7b6d2e4eb"
+          (reference "R3") (unit 1)
         )
       )
@@
     )
   )
+  (symbol (lib_id "Device:C") (at 101.6 110.49 0) (unit 1)
+    (in_bom yes) (on_board yes) (dnp no)
+    (property "Reference" "C2" (at 97.79 107.95 0)
+      (effects (font (size 1.27 1.27)) (justify left))
+    )
+    (property "Value" "C" (at 97.79 111.76 0)
+      (effects (font (size 1.27 1.27)) (justify left))
+    )
+    (property "Footprint" "Capacitor_SMD:C_0402_1005Metric" (at 102.5652 114.3 0)
+      (effects (font (size 1.27 1.27)) hide)
+    )
+    (property "Datasheet" "~" (at 101.6 110.49 0)
+      (effects (font (size 1.27 1.27)) hide)
+    )
+    (pin "1")
+    (pin "2")
+    (instances
+      (project "hx711"
+        (path "/80bd3c70-df1b-4e0c-ae87-ddc7b6d2e4eb"
+          (reference "C2") (unit 1)
+        )
+      )
+    )
+  )
   (symbol (lib_id "power:GND") (at 88.9 88.9 90) (unit 1)
-    (in_bom yes) (on_board yes) (dnp no) (fields_autoplaced)
+    (in_bom yes) (on_board yes) (dnp no)
     (property "Reference" "#PWR04" (at 95.25 88.9 0)
       (effects (font (size 1.27 1.27)) hide)
     )
-    (property "Value" "GND" (at 92.71 88.9 90)
+    (property "Value" "GND" (at 86.995 87.63 90)
       (effects (font (size 1.27 1.27)) (justify right))
     )
@@
     )
   )
+  (symbol (lib_id "power:GND") (at 101.6 114.3 0) (unit 1)
+    (in_bom yes) (on_board yes) (dnp no) (fields_autoplaced)
+    (property "Reference" "#PWR012" (at 101.6 120.65 0)
+      (effects (font (size 1.27 1.27)) hide)
+    )
+    (property "Value" "GND" (at 101.6 119.38 0)
+      (effects (font (size 1.27 1.27)))
+    )
+    (property "Footprint" "" (at 101.6 114.3 0)
+      (effects (font (size 1.27 1.27)) hide)
+    )
+    (property "Datasheet" "" (at 101.6 114.3 0)
+      (effects (font (size 1.27 1.27)) hide)
+    )
+    (pin "1")
+    (instances
+      (project "hx711"
+        (path "/80bd3c70-df1b-4e0c-ae87-ddc7b6d2e4eb"
+          (reference "#PWR012") (unit 1)
+        )
+      )
+    )
+  )
   (symbol (lib_id "Device:R") (at 105.41 48.26 90) (unit 1)
     (in_bom yes) (on_board yes) (dnp no) (fields_autoplaced)
@@
   )
   (symbol (lib_id "power:PWR_FLAG") (at 114.3 113.03 90) (unit 1)
-    (in_bom yes) (on_board yes) (dnp no) (fields_autoplaced)
+    (in_bom yes) (on_board yes) (dnp no)
     (property "Reference" "#FLG03" (at 112.395 113.03 0)
       (effects (font (size 1.27 1.27)) hide)
     )
-    (property "Value" "PWR_FLAG" (at 110.49 113.03 90)
-      (effects (font (size 1.27 1.27)) (justify left))
-    )
+    (property "Value" "PWR_FLAG" (at 109.855 119.38 0)
+      (effects (font (size 1.27 1.27)) (justify left))
+    )
