File: stm32f405rgt6/stm32f405rgt6.kicad_pcb (KiCad board)
At the start: 4 copper layers, 87.6 x 73.7 mm, 37 parts, among them J1 USART, J2 SWD, J3 I2C, J4 USB_OTG, J5 SPI, J6 AnalogInptus, SW1 SW_Push, SW2 Boot0 selector, U1 USBLC6-2SC6, U2 STM32F405RGT6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

Commit message: tweaked some stuff for the daq and added a files
Parts:
- added J7: 5V, Connector_PinHeader_1.27mm:PinHeader_1x02_P1.27mm_Vertical, F.Cu at (209.8, 111.1)
- added J7: 5V and common GND, Connector_PinHeader_1.27mm:PinHeader_1x03_P1.27mm_Vertical, F.Cu at (209.6, 81.5)
- added J8: CAN, TerminalBlock_Phoenix:TerminalBlock_Phoenix_MKDS-1,5-4_1x04_P5.00mm_Horizontal, F.Cu at (196.8, 66.5)
- added J9: 3.3V, Connector_PinHeader_1.27mm:PinHeader_1x02_P1.27mm_Vertical, F.Cu at (209.8, 116.1)
- moved J2 0.76 mm to (206.5, 88.6)
Connections:
- U2 pad 33: unconnected-(U2-PB12-Pad33) -> CAN_RX
- U2 pad 34: unconnected-(U2-PB13-Pad34) -> CAN_TX
Routing:
- net +5V: track 16.3 -> 102.9 mm
- net CAN_TX: track 0.00 -> 60.1 mm, vias 0 -> 2
- net CAN_RX: track 0.00 -> 52.1 mm, vias 0 -> 2
- net GND: track 68.1 -> 76.0 mm, vias 21 -> 26
- net +3.3V: track 30.0 -> 31.8 mm, vias 16 -> 17
- net SWO: track 54.7 -> 56.0 mm
- net unconnected-(J4-Shield-Pad6): track 19.8 -> 20.6 mm, vias 0 -> 2
- net NRST: track 108.7 -> 108.0 mm
- net SWDIO: track 39.4 -> 38.6 mm
- net SWCLK: track 43.0 -> 42.3 mm
- net SPI1_CS: track 29.9 -> 30.5 mm

Commit message: started prepping for fab
Parts:
- removed the J7 at (209.6, 81.5)
- Analog Inputs: renamed from J6
- moved J9 41.1 mm to (209.8, 74.9)
- moved J7 29.9 mm to (209.8, 81.3)
- moved J1 0.76 mm to (140.0, 132.3)
- renumbered J3 to I2C, J5 to SPI
Routing:
- net +5V: track 102.9 -> 86.9 mm
- net GND: track 76.0 -> 71.9 mm, vias 26 -> 24
Other:
- outline, holes or cut-outs redrawn
- board text added: "+"
- board text added: "-"
- board text added: "3.3V"
- board text added: "5V"
- board text added: "A0"
- board text added: "A1"
- board text added: "A2"
- board text added: "A3"
- board text added: "BOOT"
- board text added: "CAN"
- board text added: "CS"
- board text added: "GND"
- board text added: "JLCJLCJLCJLC"
- board text added: "MISO"
- board text added: "MOSI"
- board text added: "RST"
- board text added: "RUN"
- board text added: "RX"
- board text added: "SCK"
- board text added: "SCL"
- board text added: "SDA"
- board text added: "TX"
- board text added: "UART"

Commit message: added production files
Routing:
- net LinPot2: track 39.5 -> 40.8 mm
Changed lines of the file:
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@@
   (segment (start 159.512 105.788081) (end 159.512 103.187919) (width 0.25) (layer "F.Cu") (net 28))
   (segment (start 156.464 101.457685) (end 156.994315 101.988) (width 0.25) (layer "F.Cu") (net 29))
-  (segment (start 130.251 114.514) (end 128.626 112.889) (width 0.25) (layer "F.Cu") (net 29))
+  (segment (start 131.34 107.3) (end 132.19 108.15) (width 0.25) (layer "F.Cu") (net 29))
+  (segment (start 128.21 108.47) (end 129.38 107.3) (width 0.25) (layer "F.Cu") (net 29))
+  (segment (start 128.21 112.473) (end 128.21 108.47) (width 0.25) (layer "F.Cu") (net 29))
   (segment (start 156.464 101.346) (end 156.464 101.457685) (width 0.25) (layer "F.Cu") (net 29))
   (segment (start 155.702 101.2125) (end 156.3305 101.2125) (width 0.25) (layer "F.Cu") (net 29))
-  (segment (start 149.098 107.696) (end 149.352 107.95) (width 0.25) (layer "F.Cu") (net 29))
+  (segment (start 132.19 108.15) (end 149.152 108.15) (width 0.25) (layer "F.Cu") (net 29))
   (segment (start 156.994315 101.988) (end 157.835 101.988) (width 0.25) (layer "F.Cu") (net 29))
-  (segment (start 128.626 112.889) (end 128.626 108.840902) (width 0.25) (layer "F.Cu") (net 29))
   (segment (start 156.3305 101.2125) (end 156.464 101.346) (width 0.25) (layer "F.Cu") (net 29))
-  (segment (start 129.770902 107.696) (end 149.098 107.696) (width 0.25) (layer "F.Cu") (net 29))
-  (segment (start 128.626 108.840902) (end 129.770902 107.696) (width 0.25) (layer "F.Cu") (net 29))
+  (segment (start 130.251 114.514) (end 128.21 112.473) (width 0.25) (layer "F.Cu") (net 29))
+  (segment (start 129.38 107.3) (end 131.34 107.3) (width 0.25) (layer "F.Cu") (net 29))
+  (segment (start 149.152 108.15) (end 149.352 107.95) (width 0.25) (layer "F.Cu") (net 29))
   (via (at 155.702 101.2125) (size 0.8) (drill 0.4) (layers "F.Cu" "B.Cu") (net 29))
   (via (at 149.352 107.95) (size 0.8) (drill 0.4) (layers "F.Cu" "B.Cu") (net 29))
