File: stm32f405rgt6/stm32f405rgt6.kicad_sch (KiCad schematic)
At the start: 39 parts, among them J1 USART, J2 SWD, J3 I2C, J4 USB_OTG, J5 SPI, J6 AnalogInptus, J7 5V, J8 CAN, J9 3.3V, SW1 SW_Push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

Commit message: started prepping for fab
Parts:
- C1: LCSC Part # (none) -> C52923
- C10, C11: LCSC Part # (none) -> C519919
- C12, C13: LCSC Part # (none) -> C23630
- C2, C3, C4, C5, C6: LCSC Part # (none) -> C1525
- C7: LCSC Part # (none) -> C19666
- C8, C9: LCSC Part # (none) -> C15195
- D1: LCSC Part # (none) -> C72041
- J1: LCSC Part # (none) -> C5243684
- J2: LCSC Part # (none) -> C3975188
- J3, J6, J8: LCSC Part # (none) -> C2997521
- J4: LCSC Part # (none) -> C2681563
- J5: LCSC Part # (none) -> C2997523
- J7, J9: LCSC Part # (none) -> C703015
- L1: LCSC Part # (none) -> C26443
- R1, R2: LCSC Part # (none) -> C25879
- R3: LCSC Part # (none) -> C25744
- R4: LCSC Part # (none) -> C25118
- R5: LCSC Part # (none) -> C22843
- SW1: LCSC Part # (none) -> C231330
- SW2: LCSC Part # (none) -> C221841
- U1: LCSC Part # (none) -> C7519
- U2: LCSC Part # (none) -> C15742
- XC6206P332MR1: LCSC Part # (none) -> C5446
- Y1: LCSC Part # (none) -> C9006
Changed lines of the file:
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@@
   )
   (text_box "CL = ((CL1 * CL2) / (CL1 + CL2)) + Cs  where Cs = 5pf"
-    (at 19.05 188.595 0) (size 26.67 8.255)
+    (at 34.29 185.42 0) (size 26.67 8.255)
     (stroke (width 0) (type default))
     (fill (type none))
@@
       (effects (font (size 1.27 1.27)) hide)
     )
+    (property "LCSC Part #" "C15195" (at 140.335 75.565 0)
+      (effects (font (size 1.27 1.27)) hide)
+    )
     (pin "1")
     (pin "2")
@@
     )
     (property "Datasheet" "https://www.st.com/resource/en/datasheet/usblc6-2.pdf" (at 250.19 29.845 0)
+      (effects (font (size 1.27 1.27)) hide)
+    )
+    (property "LCSC Part #" "C7519" (at 245.11 38.735 0)
       (effects (font (size 1.27 1.27)) hide)
     )
@@
       (effects (font (size 1.27 1.27)) hide)
     )
+    (property "LCSC Part #" "C26443" (at 127 73.025 0)
+      (effects (font (size 1.27 1.27)) hide)
+    )
     (pin "1")
     (pin "2")
@@
       (effects (font (size 1.27 1.27)) hide)
     )
+    (property "LCSC Part #" "C25879" (at 184.15 34.925 0)
+      (effects (font (size 1.27 1.27)) hide)
+    )
     (pin "1")
     (pin "2")
@@
       (effects (font (size 1.27 1.27)) hide)
     )
+    (property "LCSC Part #" "C22843" (at 186.055 156.845 0)
+      (effects (font (size 1.27 1.27)) hide)
+    )
     (pin "1")
     (pin "2")
@@
     )
     (property "Datasheet" "~" (at 128.905 39.37 0)
+      (effects (font (size 1.27 1.27)) hide)
+    )
+    (property "LCSC Part #" "C3975188" (at 128.905 39.37 0)
       (effects (font (size 1.27 1.27)) hide)
     )
@@
       (effects (font (size 1.27 1.27)) hide)
     )
+    (property "LCSC Part #" "" (at 214.63 71.12 0)
+      (effects (font (size 1.27 1.27)) hide)
+    )
     (pin "1")
     (instances
@@
       (effects (font (size 1.27 1.27)) hide)
     )
+    (property "LCSC Part #" "C19666" (at 132.715 75.565 0)
+      (effects (font (size 1.27 1.27)) hide)
+    )
     (pin "1")
     (pin "2")
@@
       (effects (font (size 1.27 1.27)) hide)
     )
+    (property "LCSC Part #" "C25118" (at 41.91 156.21 0)
+      (effects (font (size 1.27 1.27)) hide)
+    )
     (pin "1")
     (pin "2")
@@
     )
     (property "Datasheet" "~" (at 31.75 167.64 0)
+      (effects (font (size 1.27 1.27)) hide)
+    )
+    (property "LCSC Part #" "C9006" (at 31.75 167.64 0)
       (effects (font (size 1.27 1.27)) hide)
     )
@@
       (effects (font (size 1.27 1.27)) hide)
     )
+    (property "LCSC Part #" "C52923" (at 20.955 74.93 0)
+      (effects (font (size 1.27 1.27)) hide)
+    )
     (pin "1")
     (pin "2")
@@
     )
     (property "Datasheet" "~" (at 158.75 184.785 0)
+      (effects (font (size 1.27 1.27)) hide)
+    )
+    (property "LCSC Part #" "C2997521" (at 158.75 184.785 0)
       (effects (font (size 1.27 1.27)) hide)
     )
@@
       (effects (font (size 1.27 1.27)) hide)
     )
+    (property "LCSC Part #" "C5446" (at 173.99 124.46 0)
+      (effects (font (size 1.27 1.27)) hide)
+    )
     (pin "1")
     (pin "2")
@@
       (effects (font (size 1.27 1.27)) hide)
     )
+    (property "LCSC Part #" "C1525" (at 54.61 74.93 0)
+      (effects (font (size 1.27 1.27)) hide)
+    )
     (pin "1")
     (pin "2")
@@
     )
     (property "Datasheet" "~" (at 172.72 83.82 0)
+      (effects (font (size 1.27 1.27)) hide)
+    )
+    (property "LCSC Part #" "C2997521" (at 172.72 83.82 0)
       (effects (font (size 1.27 1.27)) hide)
     )
@@
       (effects (font (size 1.27 1.27)) hide)
     )
+    (property "LCSC Part #" "C2997521" (at 162.56 40.005 0)
+      (effects (font (size 1.27 1.27)) hide)
+    )
     (pin "1")
     (pin "2")
@@
       (effects (font (size 1.27 1.27)) hide)
     )
+    (property "LCSC Part #" "C221841" (at 36.195 126.365 0)
+      (effects (font (size 1.27 1.27)) hide)
+    )
     (pin "1")
     (pin "2")
@@
     )
     (property "Datasheet" "~" (at 24.765 37.465 0)
+      (effects (font (size 1.27 1.27)) hide)
+    )
+    (property "LCSC Part #" "C5243684" (at 24.765 37.465 0)
       (effects (font (size 1.27 1.27)) hide)
     )
@@
       (effects (font (size 1.27 1.27)) hide)
     )
+    (property "LCSC Part #" "C72041" (at 177.165 154.305 0)
+      (effects (font (size 1.27 1.27)) hide)
+    )
     (pin "1")
     (pin "2")
@@
       (effects (font (size 1.27 1.27)) hide)
     )
+    (property "LCSC Part #" "C519919" (at 41.91 172.085 0)
+      (effects (font (size 1.27 1.27)) hide)
+    )
     (pin "1")
     (pin "2")
@@
       (effects (font (size 1.27 1.27)) hide)
     )
+    (property "LCSC Part #" "C1525" (at 48.895 74.93 0)
+      (effects (font (size 1.27 1.27)) hide)
+    )
     (pin "1")
     (pin "2")
@@
       (effects (font (size 1.27 1.27)) hide)
     )
+    (property "LCSC Part #" "C1525" (at 28.575 74.93 0)
+      (effects (font (size 1.27 1.27)) hide)
+    )
     (pin "1")
     (pin "2")
@@
       (effects (font (size 1.27 1.27)) hide)
     )
+    (property "LCSC Part #" "C1525" (at 35.56 74.93 0)
+      (effects (font (size 1.27 1.27)) hide)
+    )
     (pin "1")
     (pin "2")
@@
       (effects (font (size 1.27 1.27)) hide)
     )
+    (property "LCSC Part #" "" (at 214.63 78.105 0)
+      (effects (font (size 1.27 1.27)) hide)
+    )
     (pin "1")
     (instances
@@
       (effects (font (size 1.27 1.27)) hide)
     )
+    (property "LCSC Part #" "" (at 257.175 78.105 0)
+      (effects (font (size 1.27 1.27)) hide)
+    )
     (pin "1")
     (instances
@@
       (effects (font (size 1.27 1.27)) hide)
     )
+    (property "LCSC Part #" "C25744" (at 27.305 126.365 0)
+      (effects (font (size 1.27 1.27)) hide)
+    )
     (pin "1")
     (pin "2")
@@
       (effects (font (size 1.27 1.27)) hide)
     )
+    (property "LCSC Part #" "C15195" (at 35.56 102.87 0)
+      (effects (font (size 1.27 1.27)) hide)
+    )
     (pin "1")
     (pin "2")
@@
       (effects (font (size 1.27 1.27)) hide)
     )
+    (property "LCSC Part #" "C703015" (at 227.965 92.71 0)
+      (effects (font (size 1.27 1.27)) hide)
+    )
     (pin "1")
     (pin "2")
@@
     )
     (property "Datasheet" "~" (at 81.28 168.91 0)
+      (effects (font (size 1.27 1.27)) hide)
+    )
+    (property "LCSC Part #" "C23630" (at 81.28 168.91 0)
       (effects (font (size 1.27 1.27)) hide)
     )
@@
       (effects (font (size 1.27 1.27)) hide)
     )
+    (property "LCSC Part #" "" (at 257.175 70.485 0)
+      (effects (font (size 1.27 1.27)) hide)
+    )
     (pin "1")
     (instances
@@
       (effects (font (size 1.27 1.27)) hide)
     )
+    (property "LCSC Part #" "C1525" (at 42.545 74.93 0)
+      (effects (font (size 1.27 1.27)) hide)
+    )
     (pin "1")
     (pin "2")
@@
     )
     (property "Datasheet" "~" (at 188.595 34.925 0)
+      (effects (font (size 1.27 1.27)) hide)
+    )
+    (property "LCSC Part #" "C25879" (at 188.595 34.925 0)
       (effects (font (size 1.27 1.27)) hide)
     )
@@
     )
     (property "Datasheet" "https://www.st.com/resource/en/datasheet/stm32f405rg.pdf" (at 101.6 140.335 0)
+      (effects (font (size 1.27 1.27)) hide)
+    )
+    (property "LCSC Part #" "C15742" (at 101.6 140.335 0)
       (effects (font (size 1.27 1.27)) hide)
     )
@@
       (effects (font (size 1.27 1.27)) hide)
     )
+    (property "LCSC Part #" "C703015" (at 212.725 92.71 0)
+      (effects (font (size 1.27 1.27)) hide)
+    )
     (pin "1")
     (pin "2")
@@
     )
     (property "Datasheet" " ~" (at 99.695 41.91 0)
+      (effects (font (size 1.27 1.27)) hide)
+    )
+    (property "LCSC Part #" "C2681563" (at 95.885 40.64 0)
       (effects (font (size 1.27 1.27)) hide)
     )
@@
       (effects (font (size 1.27 1.27)) hide)
     )
+    (property "LCSC Part #" "C231330" (at 28.575 100.33 0)
+      (effects (font (size 1.27 1.27)) hide)
+    )
     (pin "1")
     (pin "2")
@@
       (effects (font (size 1.27 1.27)) hide)
     )
+    (property "LCSC Part #" "C23630" (at 76.2 168.91 0)
+      (effects (font (size 1.27 1.27)) hide)
+    )
     (pin "1")
     (pin "2")
@@
       (effects (font (size 1.27 1.27)) hide)
     )
+    (property "LCSC Part #" "C519919" (at 22.86 172.085 0)
+      (effects (font (size 1.27 1.27)) hide)
+    )
     (pin "1")
     (pin "2")
@@
       (effects (font (size 1.27 1.27)) hide)
     )
+    (property "LCSC Part #" "C2997523" (at 58.42 41.91 0)
+      (effects (font (size 1.27 1.27)) hide)
+    )

Commit message: added production files
Parts:
- H1, H2, H3, H4: now left out of the parts list
Changed lines of the file:
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@@
+    (stroke (width 0) (type default))
+  )
+  (polyline (pts (xy 205.74 100.33) (xy 205.74 100.965))
     (stroke (width 0) (type default))
   )
@@
   )
   (symbol (lib_id "Mechanical:MountingHole_Pad") (at 214.63 71.12 0) (unit 1)
-    (in_bom yes) (on_board yes) (dnp no) (fields_autoplaced)
+    (in_bom no) (on_board yes) (dnp no) (fields_autoplaced)
     (property "Reference" "H4" (at 217.17 68.58 0)
       (effects (font (size 1.27 1.27)) (justify left))
@@
   )
   (symbol (lib_id "Mechanical:MountingHole_Pad") (at 214.63 78.105 0) (unit 1)
-    (in_bom yes) (on_board yes) (dnp no) (fields_autoplaced)
+    (in_bom no) (on_board yes) (dnp no) (fields_autoplaced)
     (property "Reference" "H1" (at 217.17 75.565 0)
       (effects (font (size 1.27 1.27)) (justify left))
@@
   )
   (symbol (lib_id "Mechanical:MountingHole_Pad") (at 257.175 78.105 0) (unit 1)
-    (in_bom yes) (on_board yes) (dnp no) (fields_autoplaced)
+    (in_bom no) (on_board yes) (dnp no) (fields_autoplaced)
     (property "Reference" "H3" (at 259.715 75.565 0)
       (effects (font (size 1.27 1.27)) (justify left))
@@
   )
   (symbol (lib_id "Mechanical:MountingHole_Pad") (at 257.175 70.485 0) (unit 1)
-    (in_bom yes) (on_board yes) (dnp no) (fields_autoplaced)
+    (in_bom no) (on_board yes) (dnp no) (fields_autoplaced)
     (property "Reference" "H2" (at 259.715 67.945 0)
       (effects (font (size 1.27 1.27)) (justify left))
