File: STM32F030/STM32F030.kicad_sch (KiCad schematic)
At the start: 34 parts, among them J1 USB_OTG, SW1 NRST, SW2 BOOT0, U1 STM32F030RCTx, U2 MCP2200T-I-SO, U3 AZ1117-3.3, Y1 16MHz, Y2 12MHz

Commit message: finished the schematic and most of the PCB just need the PWR planes and routes
Parts:
- added D3: LED, LED_SMD:LED_0603_1608Metric, symbol Device:LED
- added R9: 2k2, Resistor_SMD:R_0603_1608Metric, symbol Device:R_Small
- C15, C16: footprint (none) -> Capacitor_SMD:C_0603_1608Metric
- U3: footprint (none) -> Package_TO_SOT_SMD:SOT-223
Connections:
- net +3.3V: now also D3.2 (A)
- net GND: now also R9.1
- new net: D3.1 (K), R9.2
Other:
- note added: "Power supply"
- note added: "values were obtained from data sheet"
- moved on the sheet: C15, C16, U3
