File: CAN IMU/CAN IMU.kicad_sch (KiCad schematic)
At the start: 4 parts, among them U1 TJA1051T, U2 AMS1117-3.3

Commit message: finished the CAN IMU schematic and pcb. Only needs some final touhces and a BOM list
Parts:
- added C10, C12, C14: 1u, Capacitor_SMD:C_0603_1608Metric_Pad1.08x0.95mm_HandSolder, symbol Device:C
- added C11, C6, C7, C8, C9: 10n, Capacitor_SMD:C_0603_1608Metric_Pad1.08x0.95mm_HandSolder, symbol Device:C
- added C13, C3: 100n, Capacitor_SMD:C_0603_1608Metric_Pad1.08x0.95mm_HandSolder, symbol Device:C
- added C4, C5: 6p, Capacitor_SMD:C_0603_1608Metric_Pad1.08x0.95mm_HandSolder, symbol Device:C
- added H1, H2, H3, H4: MountingHole, MountingHole:MountingHole_4.3mm_M4_Pad, symbol Mechanical:MountingHole
- added J1: GPIO, TerminalBlock_Phoenix:TerminalBlock_Phoenix_MKDS-1,5-3-5.08_1x03_P5.08mm_Horizontal, symbol Connector:Screw_Terminal_01x03
- added J2: ADC, TerminalBlock_Phoenix:TerminalBlock_Phoenix_MKDS-1,5-2_1x02_P5.00mm_Horizontal, symbol Connector:Screw_Terminal_01x02
- added J3: CAN, TerminalBlock_Phoenix:TerminalBlock_Phoenix_MKDS-1,5-2_1x02_P5.00mm_Horizontal, symbol Connector:Screw_Terminal_01x02
- added J4: USB_A, Connector_USB:USB_A_Molex_67643_Horizontal, symbol Connector:USB_A
- added R1: 0, Resistor_SMD:R_0603_1608Metric_Pad0.98x0.95mm_HandSolder, symbol Device:R
- added SW1: SW_Push, Button_Switch_SMD:SW_SPST_PTS645, symbol Switch:SW_Push
- added SW2: SW_SPDT, Button_Switch_SMD:SW_SPDT_PCM12, symbol Switch:SW_SPDT
- added U3: STM32F103C4Tx, Package_QFP:LQFP-48_7x7mm_P0.5mm, symbol MCU_ST_STM32F1:STM32F103C4Tx
- added x1: 8Mhz, Oscillator:Oscillator_SMD_Abracon_ASE-4Pin_3.2x2.5mm_HandSoldering, symbol Device:Crystal_GND24
- C1, C2: footprint (none) -> Capacitor_SMD:C_0603_1608Metric_Pad1.08x0.95mm_HandSolder
Connections:
- net +3.3V: now also C10.1, C11.1, C12.1, C6.1, C7.1, C8.1, C9.1, SW2.2 (B), U3.1 (VBAT), U3.24 (VDD), U3.36 (VDD), U3.48 (VDD), U3.9 (VDDA)
- net +5V: now also C13.1, C14.1, J4.1 (VBUS)
- net CAN+: now also J3.1 (Pin_1)
- net CAN-: now also J3.2 (Pin_2)
- net GND: now also U1.2 (GND), C10.2, C11.2, C12.2, C13.2, C14.2, C4.2, C5.2, C6.2, C7.2, C8.2, C9.2, J4.4 (GND), J4.5 (Shield), SW2.3 (C), U3.23 (VSS), U3.35 (VSS), U3.47 (VSS), U3.8 (VSSA)
- net CAN TX: now reaches U1.1 (TXD)
- net CAN TX: now also U3.33 (PA12)
- net CAN RX: now reaches U1.4 (RXD)
- net CAN RX: now also U3.32 (PA11)
- net CAN Silent Mode : now reaches U1.8 (S)
- net CAN Silent Mode : now also U3.34 (PA13)
- new net: C5.1, R1.2, x1.3
- new net: C3.1, SW1.1
- new net: x1.2, x1.4
- new net ADC1: J2.1 (Pin_1), U3.13 (PA3)
- new net ADC2: J2.2 (Pin_2), U3.14 (PA4)
- new net BOOT0: SW2.1 (A), U3.44 (BOOT0)
- new net GPIO1: J1.1 (Pin_1), U3.2 (PC13)
- new net GPIO2: J1.2 (Pin_2), U3.3 (PC14)
- new net GPIO3: J1.3 (Pin_3), U3.4 (PC15)
- new net HSE_IN: C4.1, U3.5 (PD0), x1.1
- new net HSE_OUT: R1.1, U3.6 (PD1)
- new net NRST: C3.2, SW1.2, U3.7 (NRST)
- no-connect marks 0 -> 29
Other:
- note added: "ADC"
- note added: "ANALOG filtering"
- note added: "BOOT0"
- note added: "CAN"
- note added: "CAN Transceiver"
- note added: "Digital Section filtering"
- note added: "GPIO"
- note added: "NRST"
- note added: "Power"
- moved on the sheet: C1, C2, U1, U2
