File: stm32f429z/CAN.kicad_sch (KiCad schematic)
At the start: 0 parts

Commit message: finished schematics and mostly finished the routing for the pcb
Parts:
- added J11, J7: CAN connector, NewMolexLibrary:Molex_MegaFit_2x03x5.70mm_Angled, symbol Connector_Generic:Conn_02x03_Top_Bottom
- added R10, R11: 120, Resistor_SMD:R_0603_1608Metric_Pad0.98x0.95mm_HandSolder, symbol Device:R_Small
- added U2, U3: TJA1051T, Package_SO:SOIC-8_3.9x4.9mm_P1.27mm, symbol Interface_CAN_LIN:TJA1051T
Connections:
- new net +5V: J11.4 (Pin_4), J7.4 (Pin_4), U2.3 (VCC), U3.3 (VCC)
- new net CAN SIlent Mode 1: U3.8 (S)
- new net CAN SIlent Mode 2: U2.8 (S)
- new net CAN1+: J11.1 (Pin_1), R11.2, U3.7 (CANH)
- new net CAN1-: J11.2 (Pin_2), R11.1, U3.6 (CANL)
- new net CAN1_RX: U3.4 (RXD)
- new net CAN1_TX: U3.1 (TXD)
- new net CAN2+: J7.1 (Pin_1), R10.2, U2.7 (CANH)
- new net CAN2-: J7.2 (Pin_2), R10.1, U2.6 (CANL)
- new net CAN2_RX: U2.4 (RXD)
- new net CAN2_TX: U2.1 (TXD)
- new net GND: J11.6 (Pin_6), J7.6 (Pin_6), U2.2 (GND), U3.2 (GND)
- no-connect marks 0 -> 4

Commit message: usb footprint changes, Silkscreen markers for pin 1 in ICs and polarity for other components. Edited excel BOM list and kicad list for BOM cost.
Parts:
- R10, R11: JLCpart# (none) -> C2906988
- U2, U3: JLCpart# (none) -> C38695
Changed lines of the file:
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@@
+      (effects (font (size 1.27 1.27)) hide)
+    )
+    (property "JLCpart#" "C38695" (at 201.93 44.45 0)
       (effects (font (size 1.27 1.27)) hide)
     )
@@
       (effects (font (size 1.27 1.27)) hide)
     )
+    (property "JLCpart#" "C38695" (at 88.9 44.45 0)
+      (effects (font (size 1.27 1.27)) hide)
+    )
     (pin "1")
     (pin "2")
@@
       (effects (font (size 1.27 1.27)) hide)
     )
+    (property "JLCpart#" "C2906988" (at 214.63 44.45 0)
+      (effects (font (size 1.27 1.27)) hide)
+    )
     (pin "1")
     (pin "2")
@@
       (effects (font (size 1.27 1.27)) hide)
     )
+    (property "JLCpart#" "" (at 246.38 44.45 0)
+      (effects (font (size 1.27 1.27)) hide)
+    )
     (pin "1")
     (pin "2")
@@
       (effects (font (size 1.27 1.27)) hide)
     )
+    (property "JLCpart#" "" (at 135.89 44.45 0)
+      (effects (font (size 1.27 1.27)) hide)
+    )
     (pin "1")
     (pin "2")
@@
       (effects (font (size 1.27 1.27)) hide)
     )
+    (property "JLCpart#" "C2906988" (at 101.6 44.45 0)
+      (effects (font (size 1.27 1.27)) hide)
+    )
