File: stm32f429z/HSE.kicad_sch (KiCad schematic)
At the start: 0 parts

Commit message: finished schematics and mostly finished the routing for the pcb
Parts:
- added C1, C2: 14pF, Capacitor_SMD:C_0603_1608Metric_Pad1.08x0.95mm_HandSolder, symbol Device:C
- added R1: 0, Resistor_SMD:R_0603_1608Metric_Pad0.98x0.95mm_HandSolder, symbol Device:R
- added X1: 16Mhz, Crystal:Crystal_SMD_3225-4Pin_3.2x2.5mm_HandSoldering, symbol Device:Crystal_GND24
Connections:
- new net: C1.1, R1.2, X1.1
- new net GND: C1.2, C2.2, X1.2, X1.4
- new net HSE_IN  : C2.1, X1.3
- new net HSE_OUT: R1.1

Commit message: usb footprint changes, Silkscreen markers for pin 1 in ICs and polarity for other components. Edited excel BOM list and kicad list for BOM cost.
Parts:
- C1, C2: JLCpart# (none) -> C5360816
- X1: JLCpart# (none) -> C12668
Changed lines of the file:
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@@
+      (effects (font (size 1.27 1.27)) hide)
+    )
+    (property "JLCpart#" "C5360816" (at 33.02 90.17 0)
       (effects (font (size 1.27 1.27)) hide)
     )
@@
     )
     (property "Datasheet" "~" (at 33.02 72.39 0)
+      (effects (font (size 1.27 1.27)) hide)
+    )
+    (property "JLCpart#" "" (at 33.02 72.39 0)
       (effects (font (size 1.27 1.27)) hide)
     )
@@
       (effects (font (size 1.27 1.27)) hide)
     )
+    (property "JLCpart#" "C5360816" (at 59.69 90.17 0)
+      (effects (font (size 1.27 1.27)) hide)
+    )
     (pin "1")
     (pin "2")
@@
       (effects (font (size 1.27 1.27)) hide)
     )
+    (property "JLCpart#" "C12668" (at 48.26 82.55 0)
+      (effects (font (size 1.27 1.27)) hide)
+    )
