File: stm32f429z/USB.kicad_sch (KiCad schematic)
At the start: 0 parts

Commit message: finished schematics and mostly finished the routing for the pcb
Parts:
- added C20: 100n, Capacitor_SMD:C_0603_1608Metric_Pad1.08x0.95mm_HandSolder, symbol Device:C
- added C21: 4.7u, Capacitor_SMD:C_0603_1608Metric_Pad1.08x0.95mm_HandSolder, symbol Device:C
- added C23: 100n, Capacitor_SMD:C_0603_1608Metric_Pad1.08x0.95mm_HandSolder, symbol Device:C_Small
- added C24, C25: 6p, Capacitor_SMD:C_0603_1608Metric_Pad1.08x0.95mm_HandSolder, symbol Device:C_Small
- added D2, D3: LED, LED_SMD:LED_0603_1608Metric_Pad1.05x0.95mm_HandSolder, symbol Device:LED
- added D6: Schottky Diode, Diode_SMD:D_0603_1608Metric_Pad1.05x0.95mm_HandSolder, symbol Device:D_Schottky
- added J13, J6: USB_OTG, Connector_USB:USB_Mini-B_Wuerth_65100516121_Horizontal, symbol Connector:USB_OTG
- added R13: 4k7, Resistor_SMD:R_0603_1608Metric_Pad0.98x0.95mm_HandSolder, symbol Device:R_Small
- added R14, R15: 2k2, Resistor_SMD:R_0603_1608Metric_Pad0.98x0.95mm_HandSolder, symbol Device:R_Small
- added U5: MCP2200T-I-SO, Package_SO:SOIC-20W_7.5x12.8mm_P1.27mm, symbol Interface_USB:MCP2200T-I-SO
- added Y1: 12MHz, Crystal:Crystal_SMD_3225-4Pin_3.2x2.5mm, symbol Device:Crystal_GND24
Connections:
- new net: D6.2 (A), J13.1 (VBUS)
- new net: R13.1, U5.4 (RST)
- new net: C25.1, U5.3 (OSC2), Y1.1
- new net: C24.1, U5.2 (OSC1), Y1.3
- new net: D3.2 (A), U5.5 (GP7/TxLED)
- new net: D2.2 (A), U5.6 (GP6/RxLED)
- new net: D2.1 (K), R14.2
- new net: D3.1 (K), R15.2
- new net +3.3V: C23.1, R13.2, U5.1 (VDD), U5.17 (V_USB)
- new net +5V: C20.1, C21.1, D6.1 (K), J6.1 (VBUS)
- new net CTS: U5.13 (CTS)
- new net GND: C20.2, C21.2, C23.2, C24.2, C25.2, J13.5 (GND), J13.6 (Shield), J6.5 (GND), J6.6 (Shield), R14.1, R15.1, U5.20 (VSS), Y1.2, Y1.4
- new net GP0: U5.16 (GP0/SSPND)
- new net GP1: U5.15 (GP1/USB-CFG)
- new net GP2: U5.14 (GP2)
- new net GP3: U5.9 (GP3)
- new net GP4: U5.8 (GP4)
- new net GP5: U5.7 (GP5)
- new net RTS: U5.11 (RTS)
- new net USART1_RX: U5.10 (TX)
- new net USART1_TX: U5.12 (RX)
- new net USB_DP+: J13.3 (D+), U5.19 (D+)
- new net USB_DP-: J13.2 (D-), U5.18 (D-)
- new net USB_OTG_FS_DP+: J6.3 (D+)
- new net USB_OTG_FS_DP-: J6.2 (D-)
- no-connect marks 0 -> 2
Other:
- note added: "CX3225GB12000D0HPQCC"
- note added: "Note: this usb will supply 5 V rather then be supplied with 5V. decoupling added to smooth power supply"
- note added: "USB OTG for data"
- note added: "USB for programming"
- note added: "USB to UART"
- note added: "differential pair is 90 ohms"

Commit message: removed alot of the silk screen, changed oscillator foor print and added GPIOs
Parts:
- Y1: footprint Crystal:Crystal_SMD_3225-4Pin_3.2x2.5mm -> Crystal:Crystal_SMD_3225-4Pin_3.2x2.5mm_HandSoldering
Changed lines of the file:
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@@
       (effects (font (size 1.27 1.27)))
     )
-    (property "Footprint" "Crystal:Crystal_SMD_3225-4Pin_3.2x2.5mm" (at 110.49 140.335 0)
+    (property "Footprint" "Crystal:Crystal_SMD_3225-4Pin_3.2x2.5mm_HandSoldering" (at 110.49 140.335 0)
       (effects (font (size 1.27 1.27)) hide)
     )

Commit message: changed some footprints, removed dimensions( was causing issues), addd a gerber filter for manufacturing(probably should be regenerated), added a BOM list
Parts:
- D6: footprint Diode_SMD:D_0603_1608Metric_Pad1.05x0.95mm_HandSolder -> Diode_SMD:D_SMA-SMB_Universal_Handsoldering
- J6: footprint Connector_USB:USB_Mini-B_Wuerth_65100516121_Horizontal -> Connector_USB:USB_A_Receptacle_GCT_USB1046
Changed lines of the file:
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@@
       (effects (font (size 1.27 1.27)))
     )
-    (property "Footprint" "Diode_SMD:D_0603_1608Metric_Pad1.05x0.95mm_HandSolder" (at 227.33 35.56 0)
+    (property "Footprint" "Diode_SMD:D_SMA-SMB_Universal_Handsoldering" (at 227.33 35.56 0)
       (effects (font (size 1.27 1.27)) hide)
     )
@@
       (effects (font (size 1.27 1.27)))
     )
-    (property "Footprint" "Connector_USB:USB_Mini-B_Wuerth_65100516121_Horizontal" (at 66.04 45.72 0)
+    (property "Footprint" "Connector_USB:USB_A_Receptacle_GCT_USB1046" (at 66.04 45.72 0)
       (effects (font (size 1.27 1.27)) hide)
     )

Commit message: usb footprint changes, Silkscreen markers for pin 1 in ICs and polarity for other components. Edited excel BOM list and kicad list for BOM cost.
Parts:
- C20, C23: JLCpart# (none) -> C76599
- C21: JLCpart# (none) -> C19666
- C24, C25: JLCpart# (none) -> C282508
- D2, D3: JLCpart# (none) -> C72038
- D6: JLCpart# (none) -> C2480
- J6: footprint Connector_USB:USB_A_Receptacle_GCT_USB1046 -> Connector_USB:USB_A_Molex_67643_Horizontal
- R13: JLCpart# (none) -> C473239
- R14, R15: JLCpart# (none) -> C427273
Changed lines of the file:
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@@
+      (effects (font (size 1.27 1.27)) hide)
+    )
+    (property "JLCpart#" "C19666" (at 111.76 48.26 0)
       (effects (font (size 1.27 1.27)) hide)
     )
@@
     )
     (property "Datasheet" " ~" (at 215.9 41.91 0)
+      (effects (font (size 1.27 1.27)) hide)
+    )
+    (property "JLCpart#" "" (at 212.09 40.64 0)
       (effects (font (size 1.27 1.27)) hide)
     )
@@
       (effects (font (size 1.27 1.27)) hide)
     )
+    (property "JLCpart#" "C473239" (at 44.45 98.425 0)
+      (effects (font (size 1.27 1.27)) hide)
+    )
     (pin "1")
     (pin "2")
@@
     )
     (property "Datasheet" "~" (at 101.6 144.145 0)
+      (effects (font (size 1.27 1.27)) hide)
+    )
+    (property "JLCpart#" "C282508" (at 101.6 144.145 0)
       (effects (font (size 1.27 1.27)) hide)
     )
@@
       (effects (font (size 1.27 1.27)) hide)
     )
+    (property "JLCpart#" "" (at 110.49 140.335 0)
+      (effects (font (size 1.27 1.27)) hide)
+    )
     (pin "1")
     (pin "2")
@@
     )
     (property "Datasheet" "http://ww1.microchip.com/downloads/en/DeviceDoc/200022228D.pdf" (at 72.39 146.05 0)
+      (effects (font (size 1.27 1.27)) hide)
+    )
+    (property "JLCpart#" "" (at 72.39 120.65 0)
       (effects (font (size 1.27 1.27)) hide)
     )
@@
       (effects (font (size 1.27 1.27)) hide)
     )
+    (property "JLCpart#" "C72038" (at 43.18 133.35 0)
+      (effects (font (size 1.27 1.27)) hide)
+    )
     (pin "1")
     (pin "2")
@@
       (effects (font (size 1.27 1.27)) hide)
     )
+    (property "JLCpart#" "C427273" (at 36.83 135.89 0)
+      (effects (font (size 1.27 1.27)) hide)
+    )
     (pin "1")
     (pin "2")
@@
       (effects (font (size 1.27 1.27)) hide)
     )
+    (property "JLCpart#" "C72038" (at 43.18 135.89 0)
+      (effects (font (size 1.27 1.27)) hide)
+    )
     (pin "1")
     (pin "2")
@@
       (effects (font (size 1.27 1.27)) hide)
     )
+    (property "JLCpart#" "C76599" (at 100.33 48.26 0)
+      (effects (font (size 1.27 1.27)) hide)
+    )
     (pin "1")
     (pin "2")
@@
     )
     (property "Datasheet" "~" (at 227.33 35.56 0)
+      (effects (font (size 1.27 1.27)) hide)
+    )
+    (property "JLCpart#" "C2480" (at 227.33 35.56 0)
       (effects (font (size 1.27 1.27)) hide)
     )
@@
       (effects (font (size 1.27 1.27)) hide)
     )
+    (property "JLCpart#" "C76599" (at 79.375 97.79 0)
+      (effects (font (size 1.27 1.27)) hide)
+    )
     (pin "1")
     (pin "2")
@@
     )
     (property "Datasheet" "~" (at 118.745 143.51 0)
+      (effects (font (size 1.27 1.27)) hide)
+    )
+    (property "JLCpart#" "C282508" (at 118.745 143.51 0)
       (effects (font (size 1.27 1.27)) hide)
     )
@@
       (effects (font (size 1.27 1.27)))
     )
-    (property "Footprint" "Connector_USB:USB_A_Receptacle_GCT_USB1046" (at 66.04 45.72 0)
+    (property "Footprint" "Connector_USB:USB_A_Molex_67643_Horizontal" (at 66.04 45.72 0)
       (effects (font (size 1.27 1.27)) hide)
     )
     (property "Datasheet" " ~" (at 66.04 45.72 0)
+      (effects (font (size 1.27 1.27)) hide)
+    )
+    (property "JLCpart#" "" (at 62.23 44.45 0)
       (effects (font (size 1.27 1.27)) hide)
     )
@@
       (effects (font (size 1.27 1.27)) hide)
     )
+    (property "JLCpart#" "C427273" (at 36.83 133.35 0)
+      (effects (font (size 1.27 1.27)) hide)
+    )

Commit message: updated some stuff
Parts:
- J6: footprint Connector_USB:USB_A_Molex_67643_Horizontal -> Connector_USB:USB_A_Wuerth_61400826021_Horizontal_Stacked
Changed lines of the file:
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@@
       (effects (font (size 1.27 1.27)))
     )
-    (property "Footprint" "Connector_USB:USB_A_Molex_67643_Horizontal" (at 66.04 45.72 0)
+    (property "Footprint" "Connector_USB:USB_A_Wuerth_61400826021_Horizontal_Stacked" (at 66.04 45.72 0)
       (effects (font (size 1.27 1.27)) hide)
     )

Commit message: something
Parts:
- J6: footprint Connector_USB:USB_A_Wuerth_61400826021_Horizontal_Stacked -> Connector_USB:USB_A_TE_292303-7_Horizontal
Changed lines of the file:
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@@
+        )
+      )
+      (project "rev2"
+        (path "/25bc3102-98ca-4c7c-b597-2d2eb7e7cb79/a8b40fa5-269b-4c25-b32b-052a9524b109"
+          (reference "C26") (unit 1)
         )
       )
@@
       (project "stm32f429z"
         (path "/09c21947-d3c4-4f82-9fb4-45f647ba61fc/a8b40fa5-269b-4c25-b32b-052a9524b109"
+          (reference "#PWR061") (unit 1)
+        )
+      )
+      (project "rev2"
+        (path "/25bc3102-98ca-4c7c-b597-2d2eb7e7cb79/a8b40fa5-269b-4c25-b32b-052a9524b109"
           (reference "#PWR061") (unit 1)
         )
@@
         )
       )
+      (project "rev2"
+        (path "/25bc3102-98ca-4c7c-b597-2d2eb7e7cb79/a8b40fa5-269b-4c25-b32b-052a9524b109"
+          (reference "J13") (unit 1)
+        )
+      )
     )
   )
@@
         )
       )
+      (project "rev2"
+        (path "/25bc3102-98ca-4c7c-b597-2d2eb7e7cb79/a8b40fa5-269b-4c25-b32b-052a9524b109"
+          (reference "R15") (unit 1)
+        )
+      )
       (project "STM32F030"
         (path "/92294cfa-b22f-416c-99d1-d973889b333f"
@@
       (project "stm32f429z"
         (path "/09c21947-d3c4-4f82-9fb4-45f647ba61fc/a8b40fa5-269b-4c25-b32b-052a9524b109"
+          (reference "#PWR060") (unit 1)
+        )
+      )
+      (project "rev2"
+        (path "/25bc3102-98ca-4c7c-b597-2d2eb7e7cb79/a8b40fa5-269b-4c25-b32b-052a9524b109"
           (reference "#PWR060") (unit 1)
         )
@@
         )
       )
+      (project "rev2"
+        (path "/25bc3102-98ca-4c7c-b597-2d2eb7e7cb79/a8b40fa5-269b-4c25-b32b-052a9524b109"
+          (reference "C25") (unit 1)
+        )
+      )
       (project "STM32F030"
         (path "/92294cfa-b22f-416c-99d1-d973889b333f"
@@
       (project "stm32f429z"
         (path "/09c21947-d3c4-4f82-9fb4-45f647ba61fc/a8b40fa5-269b-4c25-b32b-052a9524b109"
+          (reference "#PWR057") (unit 1)
+        )
+      )
+      (project "rev2"
+        (path "/25bc3102-98ca-4c7c-b597-2d2eb7e7cb79/a8b40fa5-269b-4c25-b32b-052a9524b109"
           (reference "#PWR057") (unit 1)
         )
@@
       (project "stm32f429z"
         (path "/09c21947-d3c4-4f82-9fb4-45f647ba61fc/a8b40fa5-269b-4c25-b32b-052a9524b109"
+          (reference "Y1") (unit 1)
+        )
+      )
+      (project "rev2"
+        (path "/25bc3102-98ca-4c7c-b597-2d2eb7e7cb79/a8b40fa5-269b-4c25-b32b-052a9524b109"
           (reference "Y1") (unit 1)
         )
@@
         )
       )
+      (project "rev2"
+        (path "/25bc3102-98ca-4c7c-b597-2d2eb7e7cb79/a8b40fa5-269b-4c25-b32b-052a9524b109"
+          (reference "U5") (unit 1)
+        )
+      )
       (project "STM32F030"
         (path "/92294cfa-b22f-416c-99d1-d973889b333f"
@@
         )
       )
+      (project "rev2"
+        (path "/25bc3102-98ca-4c7c-b597-2d2eb7e7cb79/a8b40fa5-269b-4c25-b32b-052a9524b109"
+          (reference "#PWR058") (unit 1)
+        )
+      )
       (project "STM32F030"
         (path "/92294cfa-b22f-416c-99d1-d973889b333f"
@@
         (path "/09c21947-d3c4-4f82-9fb4-45f647ba61fc/a8b40fa5-269b-4c25-b32b-052a9524b109"
           (reference "#PWR038") (unit 1)
+        )
+      )
+      (project "rev2"
+        (path "/25bc3102-98ca-4c7c-b597-2d2eb7e7cb79/a8b40fa5-269b-4c25-b32b-052a9524b109"
+          (reference "#PWR0104") (unit 1)
         )
       )
@@
         )
       )
+      (project "rev2"
+        (path "/25bc3102-98ca-4c7c-b597-2d2eb7e7cb79/a8b40fa5-269b-4c25-b32b-052a9524b109"
+          (reference "D2") (unit 1)
+        )
+      )
       (project "STM32F030"
         (path "/92294cfa-b22f-416c-99d1-d973889b333f"
@@
       (project "stm32f429z"
         (path "/09c21947-d3c4-4f82-9fb4-45f647ba61fc/a8b40fa5-269b-4c25-b32b-052a9524b109"
+          (reference "#PWR062") (unit 1)
+        )
+      )
+      (project "rev2"
+        (path "/25bc3102-98ca-4c7c-b597-2d2eb7e7cb79/a8b40fa5-269b-4c25-b32b-052a9524b109"
           (reference "#PWR062") (unit 1)
         )
@@
         )
       )
+      (project "rev2"
+        (path "/25bc3102-98ca-4c7c-b597-2d2eb7e7cb79/a8b40fa5-269b-4c25-b32b-052a9524b109"
+          (reference "R18") (unit 1)
+        )
+      )
       (project "STM32F030"
         (path "/92294cfa-b22f-416c-99d1-d973889b333f"
@@
         )
       )
+      (project "rev2"
+        (path "/25bc3102-98ca-4c7c-b597-2d2eb7e7cb79/a8b40fa5-269b-4c25-b32b-052a9524b109"
+          (reference "D3") (unit 1)
+        )
+      )
       (project "STM32F030"
         (path "/92294cfa-b22f-416c-99d1-d973889b333f"
@@
       (project "stm32f429z"
         (path "/09c21947-d3c4-4f82-9fb4-45f647ba61fc/a8b40fa5-269b-4c25-b32b-052a9524b109"
+          (reference "#PWR030") (unit 1)
+        )
+      )
+      (project "rev2"
+        (path "/25bc3102-98ca-4c7c-b597-2d2eb7e7cb79/a8b40fa5-269b-4c25-b32b-052a9524b109"
           (reference "#PWR030") (unit 1)
         )
@@
         )
       )
+      (project "rev2"
+        (path "/25bc3102-98ca-4c7c-b597-2d2eb7e7cb79/a8b40fa5-269b-4c25-b32b-052a9524b109"
+          (reference "C20") (unit 1)
+        )
+      )
     )
   )
@@
         )
       )
+      (project "rev2"
+        (path "/25bc3102-98ca-4c7c-b597-2d2eb7e7cb79/a8b40fa5-269b-4c25-b32b-052a9524b109"
+          (reference "#PWR029") (unit 1)
+        )
+      )
     )
   )
@@
       (project "stm32f429z"
         (path "/09c21947-d3c4-4f82-9fb4-45f647ba61fc/a8b40fa5-269b-4c25-b32b-052a9524b109"
+          (reference "D6") (unit 1)
+        )
+      )
+      (project "rev2"
+        (path "/25bc3102-98ca-4c7c-b597-2d2eb7e7cb79/a8b40fa5-269b-4c25-b32b-052a9524b109"
           (reference "D6") (unit 1)
         )
@@
         )
       )
+      (project "rev2"
+        (path "/25bc3102-98ca-4c7c-b597-2d2eb7e7cb79/a8b40fa5-269b-4c25-b32b-052a9524b109"
+          (reference "C23") (unit 1)
+        )
+      )
       (project "STM32F030"
         (path "/92294cfa-b22f-416c-99d1-d973889b333f"
@@
       (project "stm32f429z"
         (path "/09c21947-d3c4-4f82-9fb4-45f647ba61fc/a8b40fa5-269b-4c25-b32b-052a9524b109"
+          (reference "#PWR059") (unit 1)
+        )
+      )
+      (project "rev2"
+        (path "/25bc3102-98ca-4c7c-b597-2d2eb7e7cb79/a8b40fa5-269b-4c25-b32b-052a9524b109"
           (reference "#PWR059") (unit 1)
         )
@@
         )
       )
+      (project "rev2"
+        (path "/25bc3102-98ca-4c7c-b597-2d2eb7e7cb79/a8b40fa5-269b-4c25-b32b-052a9524b109"
+          (reference "C24") (unit 1)
+        )
+      )
       (project "STM32F030"
         (path "/92294cfa-b22f-416c-99d1-d973889b333f"
@@
         )
       )
+      (project "rev2"
+        (path "/25bc3102-98ca-4c7c-b597-2d2eb7e7cb79/a8b40fa5-269b-4c25-b32b-052a9524b109"
+          (reference "#PWR0102") (unit 1)
+        )
+      )
     )
   )
@@
       (effects (font (size 1.27 1.27)))
     )
-    (property "Footprint" "Connector_USB:USB_A_Wuerth_61400826021_Horizontal_Stacked" (at 66.04 45.72 0)
+    (property "Footprint" "Connector_USB:USB_A_TE_292303-7_Horizontal" (at 66.04 45.72 0)
       (effects (font (size 1.27 1.27)) hide)
     )
@@
         )
       )
+      (project "rev2"
+        (path "/25bc3102-98ca-4c7c-b597-2d2eb7e7cb79/a8b40fa5-269b-4c25-b32b-052a9524b109"
+          (reference "J6") (unit 1)
+        )
+      )
     )
   )
@@
       (project "stm32f429z"
         (path "/09c21947-d3c4-4f82-9fb4-45f647ba61fc/a8b40fa5-269b-4c25-b32b-052a9524b109"
+          (reference "#PWR063") (unit 1)
+        )
+      )
+      (project "rev2"
+        (path "/25bc3102-98ca-4c7c-b597-2d2eb7e7cb79/a8b40fa5-269b-4c25-b32b-052a9524b109"
           (reference "#PWR063") (unit 1)
         )
@@
         )
       )
+      (project "rev2"
+        (path "/25bc3102-98ca-4c7c-b597-2d2eb7e7cb79/a8b40fa5-269b-4c25-b32b-052a9524b109"
+          (reference "R14") (unit 1)
+        )
+      )
       (project "STM32F030"
         (path "/92294cfa-b22f-416c-99d1-d973889b333f"
@@
         )
       )
+      (project "rev2"
+        (path "/25bc3102-98ca-4c7c-b597-2d2eb7e7cb79/a8b40fa5-269b-4c25-b32b-052a9524b109"
+          (reference "#PWR0105") (unit 1)
+        )
+      )
     )
   )
@@
         )
       )
+      (project "rev2"
+        (path "/25bc3102-98ca-4c7c-b597-2d2eb7e7cb79/a8b40fa5-269b-4c25-b32b-052a9524b109"
+          (reference "#PWR056") (unit 1)
+        )
+      )
       (project "STM32F030"
         (path "/92294cfa-b22f-416c-99d1-d973889b333f"
@@
         )
       )
+      (project "rev2"
+        (path "/25bc3102-98ca-4c7c-b597-2d2eb7e7cb79/a8b40fa5-269b-4c25-b32b-052a9524b109"
+          (reference "#PWR0103") (unit 1)
+        )
+      )
