File: stm32f429z/connectors.kicad_sch (KiCad schematic)
At the start: 23 parts, among them J1 ADC connector 2, J10 UART 1 connectors, J12 USB to UART GPIO, J14 I2C 1 connector, J15 GPIO, J16 GPIO, J2 ADC connector 1, J3 SPI 2 connector, J4 SPI 1 connector, J5 I2C 2 connector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

Commit message: usb footprint changes, Silkscreen markers for pin 1 in ICs and polarity for other components. Edited excel BOM list and kicad list for BOM cost.
Parts:
- C19: JLCpart# (none) -> C124567
- C28: JLCpart# (none) -> C76599
- R12: JLCpart# (none) -> C4226066
- R2, R3, R4, R5: JLCpart# (none) -> C441885
- R6, R7, R8, R9: JLCpart# (none) -> C427273
Changed lines of the file:
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@@
+      (effects (font (size 1.27 1.27)) hide)
+    )
+    (property "JLCpart#" "C4226066" (at 180.975 132.715 0)
       (effects (font (size 1.27 1.27)) hide)
     )
@@
     )
     (property "Datasheet" "~" (at 227.965 146.05 0)
+      (effects (font (size 1.27 1.27)) hide)
+    )
+    (property "JLCpart#" "" (at 227.965 146.05 0)
       (effects (font (size 1.27 1.27)) hide)
     )
@@
       (effects (font (size 1.27 1.27)) hide)
     )
+    (property "JLCpart#" "C427273" (at 46.99 99.06 0)
+      (effects (font (size 1.27 1.27)) hide)
+    )
     (pin "1")
     (pin "2")
@@
     )
     (property "Datasheet" "~" (at 66.04 105.41 0)
+      (effects (font (size 1.27 1.27)) hide)
+    )
+    (property "JLCpart#" "" (at 66.04 105.41 0)
       (effects (font (size 1.27 1.27)) hide)
     )
@@
       (effects (font (size 1.27 1.27)) hide)
     )
+    (property "JLCpart#" "C76599" (at 180.975 142.875 0)
+      (effects (font (size 1.27 1.27)) hide)
+    )
     (pin "1")
     (pin "2")
@@
       (effects (font (size 1.27 1.27)) hide)
     )
+    (property "JLCpart#" "C441885" (at 224.79 36.83 0)
+      (effects (font (size 1.27 1.27)) hide)
+    )
     (pin "1")
     (pin "2")
@@
     )
     (property "Datasheet" "~" (at 157.48 49.53 0)
+      (effects (font (size 1.27 1.27)) hide)
+    )
+    (property "JLCpart#" "" (at 157.48 49.53 0)
       (effects (font (size 1.27 1.27)) hide)
     )
@@
       (effects (font (size 1.27 1.27)) hide)
     )
+    (property "JLCpart#" "C124567" (at 196.85 36.83 0)
+      (effects (font (size 1.27 1.27)) hide)
+    )
     (pin "1")
     (pin "2")
@@
     )
     (property "Datasheet" "~" (at 45.72 63.5 0)
+      (effects (font (size 1.27 1.27)) hide)
+    )
+    (property "JLCpart#" "" (at 45.72 63.5 0)
       (effects (font (size 1.27 1.27)) hide)
     )
@@
       (effects (font (size 1.27 1.27)) hide)
     )
+    (property "JLCpart#" "C427273" (at 124.46 99.06 0)
+      (effects (font (size 1.27 1.27)) hide)
+    )
     (pin "1")
     (pin "2")
@@
     )
     (property "Datasheet" "~" (at 45.72 43.18 0)
+      (effects (font (size 1.27 1.27)) hide)
+    )
+    (property "JLCpart#" "" (at 45.72 43.18 0)
       (effects (font (size 1.27 1.27)) hide)
     )
@@
       (effects (font (size 1.27 1.27)) hide)
     )
+    (property "JLCpart#" "" (at 102.87 49.53 0)
+      (effects (font (size 1.27 1.27)) hide)
+    )
     (pin "1")
     (pin "2")
@@
     )
     (property "Datasheet" "~" (at 210.82 36.83 0)
+      (effects (font (size 1.27 1.27)) hide)
+    )
+    (property "JLCpart#" "" (at 210.82 36.83 0)
       (effects (font (size 1.27 1.27)) hide)
     )
@@
       (effects (font (size 1.27 1.27)) hide)
     )
+    (property "JLCpart#" "" (at 125.73 138.43 0)
+      (effects (font (size 1.27 1.27)) hide)
+    )
     (pin "1")
     (pin "2")
@@
       (effects (font (size 1.27 1.27)) hide)
     )
+    (property "JLCpart#" "C441885" (at 224.79 41.91 0)
+      (effects (font (size 1.27 1.27)) hide)
+    )
     (pin "1")
     (pin "2")
@@
     )
     (property "Datasheet" "~" (at 227.965 132.08 0)
+      (effects (font (size 1.27 1.27)) hide)
+    )
+    (property "JLCpart#" "" (at 227.965 132.08 0)
       (effects (font (size 1.27 1.27)) hide)
     )
@@
       (effects (font (size 1.27 1.27)) hide)
     )
+    (property "JLCpart#" "C427273" (at 132.08 104.14 0)
+      (effects (font (size 1.27 1.27)) hide)
+    )
     (pin "1")
     (pin "2")
@@
       (effects (font (size 1.27 1.27)) hide)
     )
+    (property "JLCpart#" "" (at 170.18 139.065 0)
+      (effects (font (size 1.27 1.27)) hide)
+    )
     (pin "1")
     (pin "2")
@@
       (effects (font (size 1.27 1.27)) hide)
     )
+    (property "JLCpart#" "C441885" (at 224.79 31.75 0)
+      (effects (font (size 1.27 1.27)) hide)
+    )
     (pin "1")
     (pin "2")
@@
       (effects (font (size 1.27 1.27)) hide)
     )
+    (property "JLCpart#" "C441885" (at 224.79 34.29 0)
+      (effects (font (size 1.27 1.27)) hide)
+    )
     (pin "1")
     (pin "2")
@@
     )
     (property "Datasheet" "~" (at 52.07 140.97 0)
+      (effects (font (size 1.27 1.27)) hide)
+    )
+    (property "JLCpart#" "" (at 52.07 140.97 0)
       (effects (font (size 1.27 1.27)) hide)
     )
@@
       (effects (font (size 1.27 1.27)) hide)
     )
+    (property "JLCpart#" "C427273" (at 54.61 104.14 0)
+      (effects (font (size 1.27 1.27)) hide)
+    )
     (pin "1")
     (pin "2")
@@
       (effects (font (size 1.27 1.27)) hide)
     )
+    (property "JLCpart#" "" (at 143.51 105.41 0)
+      (effects (font (size 1.27 1.27)) hide)
+    )

Commit message: something
Parts:
- J15, J16: footprint TerminalBlock_Phoenix:TerminalBlock_Phoenix_MKDS-1,5-5_1x05_P5.00mm_Horizontal -> TerminalBlock_Phoenix:TerminalBlock_Phoenix_MPT-0,5-5-2.54_1x05_P2.54mm_Horizontal
