File: rev2/rev2.kicad_sch (KiCad schematic)
At the start: 52 parts, among them J1 Termination, J10 GPIO, J2 CAN1, J3 Termination, J4 CAN2, J5 SWD ASYNC, J6 LIN Pots, J7 AIN, J8 USB_OTG, J9 PWR_USB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

Commit message: tweaked the differential traces and made thhem compliant to JLC04161H-7628 guidlines for controlled impedance. Also I think I might remove the 10 pin header for SWD/JTAG in favor of just SWD to safe on space.
Parts:
- R2, R6, R7, R8: value 100 -> 0
Changed lines of the file:
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@@
     (effects (font (size 1.27 1.27)) (justify left top))
   )
+  (text_box "Using 0 ohm resistors to jump the SWD/JTAG connector. If for whatever reason a current limiting resistor is needed for the connector they can be added."
+    (at 363.22 59.69 0) (size 36.83 12.7)
+    (stroke (width 0) (type default))
+    (fill (type none))
+    (effects (font (size 1.27 1.27)) (justify left top))
+  )
   (text_box "Equation used to calculate CL1 and CL2 is \n(Cl1 * Cl2) / (Cl1 +cl2)  + cs where cs = 5pf and cl1 = cl2\n"
     (at 97.79 150.495 0) (size 66.675 6.35)
@@
     (effects (font (size 1.27 1.27)) (justify left top))
   )
+  (text_box "Address is configurable with SDO/SA0 pin( pin 1). setting this pin LOW sets address to 6A. If pin is set HIGH then the address is 6B NOTE: these are the 7-bit addresses in most cases to use them you need to shift the adress 1 bit to the left."
+    (at 356.87 168.91 0) (size 46.99 15.24)
+    (stroke (width 0) (type default))
+    (fill (type none))
+    (effects (font (size 1.27 1.27)) (justify left top))
+  )
   (text_box "I decoupling capacitors is used for each VDD/VBAT pin present plus a bulk decoupling capacitor\n"
     (at 104.775 17.145 0) (size 32.385 10.16)
@@
       (effects (font (size 1.27 1.27)))
     )
-    (property "Value" "100" (at 370.84 79.375 90)
+    (property "Value" "0" (at 370.84 79.375 90)
       (effects (font (size 1.27 1.27)))
     )
@@
       (effects (font (size 1.27 1.27)))
     )
-    (property "Value" "100" (at 370.84 74.295 90)
+    (property "Value" "0" (at 370.84 74.295 90)
       (effects (font (size 1.27 1.27)))
     )
@@
       (effects (font (size 1.27 1.27)))
     )
-    (property "Value" "100" (at 370.84 84.455 90)
+    (property "Value" "0" (at 370.84 84.455 90)
       (effects (font (size 1.27 1.27)))
     )
@@
       (effects (font (size 1.27 1.27)))
     )
-    (property "Value" "100" (at 370.84 76.835 90)
+    (property "Value" "0" (at 370.84 76.835 90)
       (effects (font (size 1.27 1.27)))
     )

Commit message: removed the 10 pin SWD/JTAG header in favor of just a 3 pin SWD connector.in addition, also added a 3.3V and a 5V header for external power supplies
Parts:
- removed C25: 500n, Capacitor_SMD:C_0603_1608Metric_Pad1.08x0.95mm_HandSolder, symbol Device:C
- removed J5: SWD ASYNC, Connector_PinHeader_2.54mm:PinHeader_2x05_P2.54mm_Vertical, symbol Connector_Generic:Conn_02x05_Odd_Even
- removed R2, R6, R7, R8: 0, Resistor_SMD:R_0603_1608Metric_Pad0.98x0.95mm_HandSolder, symbol Device:R_Small
- added J11: SWD, Connector_PinHeader_2.54mm:PinHeader_1x03_P2.54mm_Vertical, symbol Connector:Conn_01x03_Pin
- added J12: 5V power breakout, Connector_PinHeader_2.54mm:PinHeader_1x02_P2.54mm_Vertical, symbol Connector:Conn_01x02_Pin
- added J5: 3.3V power breakout, Connector_PinHeader_2.54mm:PinHeader_1x02_P2.54mm_Vertical, symbol Connector:Conn_01x02_Pin
Connections:
- net +3.3V: now also J5.1 (Pin_1)
- net +5V: now also J12.1 (Pin_1)
- net GND: now also J11.3 (Pin_3), J12.2 (Pin_2), J5.2 (Pin_2)
- net SYS_JTCK_SWCLK: now also J11.2 (Pin_2)
- net SYS_JTMS_SWDIO: now also J11.1 (Pin_1)
- no-connect marks 87 -> 85
