File: Rev2.2/Rev2.2.kicad_sch (KiCad schematic)
At the start: 30 parts, among them J1 Termination, J10 USART1, J12 5V power breakout, J15 USART6, J2 CAN1, J3 Termination, J4 CAN2, J5 3.3V power breakout, J7 GPIO1, U1 STM32F429ZITx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

Commit message: added labels that tell you which pins the connectors are connected to for analog, GPIO, and LEDs. Also added a label for the USB C connector called Power to indicate its function
Changed lines of the file:
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@@
     )
   )
-  (text_box "max current is plus of minus 20mA\n"
+  (text_box "max current is plus or minus 20mA\n"
     (at 154.94 142.875 0) (size 22.225 6.35)
     (stroke (width 0) (type default))
