File: ESC/PWM_polarity.kicad_sch (KiCad schematic)
At the start: 4 parts, among them U3 74AHC04

Commit message: finished first mock up of the esc scheamtic still need to check everything works tho
Parts:
- C11, C12: footprint (none) -> Capacitor_SMD:C_0603_1608Metric_Pad1.08x0.95mm_HandSolder
Changed lines of the file:
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@@
       (effects (font (size 1.27 1.27)) (justify left))
     )
-    (property "Footprint" "" (at 123.5202 36.195 0)
+    (property "Footprint" "Capacitor_SMD:C_0603_1608Metric_Pad1.08x0.95mm_HandSolder" (at 123.5202 36.195 0)
       (effects (font (size 1.27 1.27)) hide)
     )
@@
       (effects (font (size 1.27 1.27)) (justify left))
     )
-    (property "Footprint" "" (at 260.0452 36.195 0)
+    (property "Footprint" "Capacitor_SMD:C_0603_1608Metric_Pad1.08x0.95mm_HandSolder" (at 260.0452 36.195 0)
       (effects (font (size 1.27 1.27)) hide)
     )
