File: tubeScreamer/tubeScreamer.kicad_sch (KiCad schematic)
At the start: 42 parts, among them J1 IN, J2 Power, J3 AudioJack2, Q1 2SC1815, Q2 2SC1815, U1 Opamp_Dual, U2 Opamp_Dual

Commit message: added values to some components that i forgot to add
Parts:
- C9: value C -> 1u
- R14: value R -> 1k
Changed lines of the file:
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@@
       (effects (font (size 1.27 1.27)))
     )
-    (property "Value" "R" (at 219.075 101.6 90)
+    (property "Value" "1k" (at 219.075 101.6 90)
       (effects (font (size 1.27 1.27)))
     )
@@
       (effects (font (size 1.27 1.27)))
     )
-    (property "Value" "C" (at 206.375 100.33 90)
-      (effects (font (size 1.27 1.27)))
-    )
+    (property "Value" "1u" (at 206.375 100.33 90)
+      (effects (font (size 1.27 1.27)))
+    )
