File: Delay/Delay.kicad_sch (KiCad schematic)
At the start: 28 parts, among them J1 AudioJack2, J2 9V input, U1 PT2399, U2 KF50BDT, U3 TL072

Commit message: added another op amp to the delay
Parts:
- added C14: 100n, symbol Device:C_Small
- added U4: TL072, symbol Amplifier_Operational:TL072
Connections:
- net 4.5V: now also C14.2
- net GND: now also J1.S
- net at J1.T: now also C14.1; no longer U3.2 (-)
- net at U3.1: now also U3.2 (-), U4.3 (+)
- new net: U4.1, U4.2 (-)
Other:
- note added: "4.5V offsett added to the signal"
- note added: "Delay IC ( PT2399 )"
- note added: "Input buffer"
- note added: "coupling cap"
- moved on the sheet: J1
Changed lines of the file:
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@@
   (junction (at 34.29 97.79) (diameter 0) (color 0 0 0 0)
   )
+  (junction (at 46.99 43.18) (diameter 0) (color 0 0 0 0)
+  )
+  (junction (at 74.93 45.72) (diameter 0) (color 0 0 0 0)
+  )
   (junction (at 147.32 83.82) (diameter 0) (color 0 0 0 0)
   )
@@
     (stroke (width 0) (type default))
   )
+  (wire (pts (xy 112.395 55.88) (xy 136.525 55.88))
+    (stroke (width 0) (type default))
+  )
   (wire (pts (xy 147.32 91.44) (xy 140.97 91.44))
     (stroke (width 0) (type default))
@@
     (stroke (width 0) (type default))
   )
+  (wire (pts (xy 38.1 43.18) (xy 46.99 43.18))
+    (stroke (width 0) (type default))
+  )
   (wire (pts (xy 38.1 91.44) (xy 38.1 92.71))
     (stroke (width 0) (type default))
@@
     (stroke (width 0) (type default))
   )
+  (wire (pts (xy 74.93 45.72) (xy 69.85 45.72))
+    (stroke (width 0) (type default))
+  )
   (wire (pts (xy 109.22 87.63) (xy 115.57 87.63))
     (stroke (width 0) (type default))
   )
+  (wire (pts (xy 27.305 40.64) (xy 27.305 26.035))
+    (stroke (width 0) (type default))
+  )
+  (wire (pts (xy 46.99 43.18) (xy 54.61 43.18))
+    (stroke (width 0) (type default))
+  )
+  (wire (pts (xy 74.93 45.72) (xy 115.57 45.72))
+    (stroke (width 0) (type default))
+  )
   (wire (pts (xy 85.09 85.09) (xy 93.98 85.09))
     (stroke (width 0) (type default))
@@
     (stroke (width 0) (type default))
   )
+  (wire (pts (xy 112.395 55.88) (xy 112.395 50.8))
+    (stroke (width 0) (type default))
+  )
   (wire (pts (xy 34.29 91.44) (xy 34.29 92.71))
     (stroke (width 0) (type default))
@@
     (stroke (width 0) (type default))
   )
+  (wire (pts (xy 49.53 48.26) (xy 49.53 53.34))
+    (stroke (width 0) (type default))
+  )
+  (wire (pts (xy 130.81 48.26) (xy 136.525 48.26))
+    (stroke (width 0) (type default))
+  )
   (wire (pts (xy 34.29 90.17) (xy 34.29 91.44))
     (stroke (width 0) (type default))
@@
     (stroke (width 0) (type default))
   )
+  (wire (pts (xy 49.53 53.34) (xy 74.93 53.34))
+    (stroke (width 0) (type default))
+  )
   (wire (pts (xy 140.97 83.82) (xy 140.97 85.09))
     (stroke (width 0) (type default))
@@
     (stroke (width 0) (type default))
   )
+  (wire (pts (xy 112.395 50.8) (xy 115.57 50.8))
+    (stroke (width 0) (type default))
+  )
   (wire (pts (xy 147.32 83.82) (xy 153.67 83.82))
     (stroke (width 0) (type default))
@@
     (stroke (width 0) (type default))
   )
+  (wire (pts (xy 136.525 48.26) (xy 136.525 55.88))
+    (stroke (width 0) (type default))
+  )
   (wire (pts (xy 140.97 91.44) (xy 140.97 92.71))
     (stroke (width 0) (type default))
@@
     (stroke (width 0) (type default))
   )
+  (wire (pts (xy 27.305 43.18) (xy 33.02 43.18))
+    (stroke (width 0) (type default))
+  )
   (wire (pts (xy 34.29 99.06) (xy 34.29 97.79))
     (stroke (width 0) (type default))
   )
+  (wire (pts (xy 54.61 48.26) (xy 49.53 48.26))
+    (stroke (width 0) (type default))
+  )
+  (wire (pts (xy 27.305 26.035) (xy 16.51 26.035))
+    (stroke (width 0) (type default))
+  )
   (wire (pts (xy 105.41 115.57) (xy 105.41 116.84))
     (stroke (width 0) (type default))
@@
     (stroke (width 0) (type default))
   )
-  (wire (pts (xy 29.21 48.26) (xy 54.61 48.26))
-    (stroke (width 0) (type default))
-  )
   (wire (pts (xy 48.26 85.09) (xy 55.88 85.09))
     (stroke (width 0) (type default))
@@
     (stroke (width 0) (type default))
   )
+  (wire (pts (xy 74.93 53.34) (xy 74.93 45.72))
+    (stroke (width 0) (type default))
+  )
   (wire (pts (xy 113.03 102.87) (xy 115.57 102.87))
     (stroke (width 0) (type default))
@@
     (stroke (width 0) (type default))
   )
+  (wire (pts (xy 46.99 40.005) (xy 46.99 43.18))
+    (stroke (width 0) (type default))
+  )
   (wire (pts (xy 147.32 91.44) (xy 147.32 90.17))
     (stroke (width 0) (type default))
@@
     (stroke (width 0) (type default))
   )
+  (rectangle (start 92.075 69.85) (end 172.72 124.46)
+    (stroke (width 0) (type default))
+    (fill (type none))
+  )
   (rectangle (start 13.97 69.85) (end 88.9 107.95)
     (stroke (width 0) (type default))
@@
     (effects (font (size 1.27 1.27)) (justify left top))
   )
+  (text "4.5V offsett added to the signal\n" (at 32.385 31.115 0)
+    (effects (font (size 1.27 1.27)) (justify left bottom))
+  )
+  (text "coupling cap\n" (at 29.845 47.625 0)
+    (effects (font (size 1.27 1.27)) (justify left bottom))
+  )
+  (text "Delay IC ( PT2399 )\n" (at 121.92 73.025 0)
+    (effects (font (size 1.27 1.27)) (justify left bottom))
+  )
   (text "https://www.mouser.com/ProductDetail/STMicroelectronics/KF50BDT-TR?qs=Tj7OqeScv5LVEpfIzte25Q%3D%3D"
     (at 38.1 107.95 0)
@@
     (effects (font (size 2 2)) (justify left bottom))
   )
+  (text "Input buffer\n" (at 55.245 57.785 0)
+    (effects (font (size 1.27 1.27)) (justify left bottom))
+  )
   (text "VCO time table" (at 40.64 148.59 0)
     (effects (font (size 1.27 1.27)) (justify left bottom))
@@
     )
   )
-  (global_label "4.5V" (shape input) (at 54.61 43.18 180) (fields_autoplaced)
-    (effects (font (size 1.27 1.27)) (justify right))
-    (property "Intersheetrefs" "${INTERSHEET_REFS}" (at 47.5124 43.18 0)
-      (effects (font (size 1.27 1.27)) (justify right) hide)
+  (global_label "4.5V" (shape input) (at 46.99 40.005 90) (fields_autoplaced)
+    (effects (font (size 1.27 1.27)) (justify left))
+    (property "Intersheetrefs" "${INTERSHEET_REFS}" (at 46.99 32.9074 90)
+      (effects (font (size 1.27 1.27)) (justify left) hide)
     )
   )
@@
     )
   )
+  (symbol (lib_id "Device:C_Small") (at 35.56 43.18 90) (unit 1)
+    (in_bom yes) (on_board yes) (dnp no) (fields_autoplaced)
+    (property "Reference" "C14" (at 35.5663 36.83 90)
+      (effects (font (size 1.27 1.27)))
+    )
+    (property "Value" "100n" (at 35.5663 39.37 90)
+      (effects (font (size 1.27 1.27)))
+    )
+    (property "Footprint" "" (at 35.56 43.18 0)
+      (effects (font (size 1.27 1.27)) hide)
+    )
+    (property "Datasheet" "~" (at 35.56 43.18 0)
+      (effects (font (size 1.27 1.27)) hide)
+    )
+    (pin "1")
+    (pin "2")
+    (instances
+      (project "Delay"
+        (path "/86c4b405-e748-4cf6-bcf3-b45a2fb6ae9f"
+          (reference "C14") (unit 1)
+        )
+      )
+    )
+  )
   (symbol (lib_id "Device:C_Small") (at 77.47 90.17 0) (unit 1)
     (in_bom yes) (on_board yes) (dnp no) (fields_autoplaced)
@@
     )
   )
-  (symbol (lib_id "Connector_Audio:AudioJack2") (at 24.13 48.26 0) (unit 1)
+  (symbol (lib_id "Connector_Audio:AudioJack2") (at 22.225 43.18 0) (unit 1)
     (in_bom yes) (on_board yes) (dnp no) (fields_autoplaced)
-    (property "Reference" "J1" (at 23.495 39.37 0)
+    (property "Reference" "J1" (at 21.59 34.29 0)
       (effects (font (size 1.27 1.27)))
     )
-    (property "Value" "AudioJack2" (at 23.495 41.91 0)
+    (property "Value" "AudioJack2" (at 21.59 36.83 0)
       (effects (font (size 1.27 1.27)))
     )
-    (property "Footprint" "" (at 24.13 48.26 0)
+    (property "Footprint" "" (at 22.225 43.18 0)
       (effects (font (size 1.27 1.27)) hide)
     )
-    (property "Datasheet" "~" (at 24.13 48.26 0)
+    (property "Datasheet" "~" (at 22.225 43.18 0)
       (effects (font (size 1.27 1.27)) hide)
     )
@@
     )
   )
+  (symbol (lib_id "Amplifier_Operational:TL072") (at 123.19 48.26 0) (unit 1)
+    (in_bom yes) (on_board yes) (dnp no) (fields_autoplaced)
+    (property "Reference" "U4" (at 123.19 38.1 0)
+      (effects (font (size 1.27 1.27)))
+    )
+    (property "Value" "TL072" (at 123.19 40.64 0)
+      (effects (font (size 1.27 1.27)))
+    )
+    (property "Footprint" "" (at 123.19 48.26 0)
+      (effects (font (size 1.27 1.27)) hide)
+    )
+    (property "Datasheet" "http://www.ti.com/lit/ds/symlink/tl071.pdf" (at 123.19 48.26 0)
+      (effects (font (size 1.27 1.27)) hide)
+    )
+    (pin "1")
+    (pin "2")
+    (pin "3")
+    (pin "5")
+    (pin "6")
+    (pin "7")
+    (pin "4")
+    (pin "8")
+    (instances
+      (project "Delay"
+        (path "/86c4b405-e748-4cf6-bcf3-b45a2fb6ae9f"
+          (reference "U4") (unit 1)
+        )
+      )
+    )
+  )
   (symbol (lib_id "Regulator_Linear:KF50BDT") (at 63.5 85.09 0) (unit 1)
     (in_bom yes) (on_board yes) (dnp no) (fields_autoplaced)
@@
         )
       )
+    )
+  )
+  (symbol (lib_id "power:GND") (at 16.51 26.035 0) (unit 1)
+    (in_bom yes) (on_board yes) (dnp no) (fields_autoplaced)
+    (property "Reference" "#PWR012" (at 16.51 32.385 0)
+      (effects (font (size 1.27 1.27)) hide)
+    )
+    (property "Value" "GND" (at 16.51 30.48 0)
+      (effects (font (size 1.27 1.27)))
+    )
+    (property "Footprint" "" (at 16.51 26.035 0)
+      (effects (font (size 1.27 1.27)) hide)
+    )
+    (property "Datasheet" "" (at 16.51 26.035 0)
+      (effects (font (size 1.27 1.27)) hide)
+    )
+    (pin "1")
+    (instances
+      (project "Delay"
+        (path "/86c4b405-e748-4cf6-bcf3-b45a2fb6ae9f"
+          (reference "#PWR012") (unit 1)
+        )
+      )

Commit message: finished the schematic
Parts:
- removed U4: TL072, symbol Amplifier_Operational:TL072
- added C15: 47p, symbol Device:C
- added C16, C18, C24: 1u, symbol Device:C
- added C17: 100p, symbol Device:C
- added C19: 4700p, symbol Device:C_Small
- added C20: 0.022u, symbol Device:C_Small
- added C21: 0.047u, symbol Device:C_Small
- added C22: 1u, symbol Device:C_Small
- added C23: 0.01u, symbol Device:C_Small
- added J3: CLK_OUT_TST, symbol Connector:Conn_01x01_Pin
- added J4: AudioJack2, symbol Connector_Audio:AudioJack2
- added R10: 180k, symbol Device:R
- added R11: 360k, symbol Device:R
- added R12: 22k, symbol Device:R_Small
- added R13: 10k, symbol Device:R
- added R14: 12k, symbol Device:R
- added R15: 1k, symbol Device:R
- added R16: 100k, symbol Device:R
- added R17: 5k1, symbol Device:R_Small
- added R18: 2k, symbol Device:R_Small
- added R19: 20k, symbol Device:R_Small
- added RV2, RV3, RV4: 20k?, symbol Device:R_Potentiometer_Small
- added unit 2 of U3
- added unit 3 of U3
- J2: value 9V input -> 9V input
- R1: value 10 -> 2k7
Connections:
- net +9V: now also U3.8 (V+)
- net 4.5V: now also U3.5 (+); no longer C14.2
- net GND: now also C19.2, C21.2, C23.2, J4.S, R16.2, RV3.1, RV4.1, U3.4 (V-)
- net at R5.2: now also R6.2, C19.1, R13.2, R17.1
- net at U3.1: now also C15.2, C16.1, R11.2, R12.1; no longer U3.2 (-)
- net at R7.2: now also C23.1, C24.1
- net at U1.5 (CLK_O): now also J3.1 (Pin_1)
- new net: C21.1, R18.2, RV3.2
- new net: C14.2, R10.1
- new net: C16.2, R13.1
- new net: C15.1, R10.2, R11.1, U3.2 (-)
- new net: C18.2, R15.1
- new net: J4.T, R15.2, R16.1
- new net: C20.2, RV3.3
- new net: C17.2, C18.1, R14.2, U3.7
- new net: R12.2, RV2.1, RV2.2
- new net: C17.1, R14.1, R19.1, RV2.3, U3.6 (-)
- new net: C24.2, R18.1, RV4.3
- new net: C20.1, R17.2
- new net: C22.2, RV4.2
- new net: C22.1, R19.2
- no-connect marks 1 -> 0
Other:
- note added: "4.5V centers signal to 4.5"
- note added: "Op amp power"
- note added: "high pass filter Fc = 1.59 hz"
- note added: "high pass filter to filter out DC Fc = 4 hz"
- note added: "level"
- note added: "output buffer"
- note added: "repeats"
- note removed: "4.5V offsett added to the signal"
- note removed: "coupling cap"
- moved on the sheet: C1, C10, C11, C12, C13, C14, C2, C3, C4, C5, C6, C7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
