File: OpAmpDistortion/OpAmpDistortion.kicad_pcb (KiCad board)
At the start: 2 copper layers, 31.4 x 18.2 mm, 20 parts, among them J1 INPUT, J2 OUTPUT, U1 NE5532

Commit message: editied the PCB
Parts:
- moved RV2 0.11 mm to (152.6, 88.4)
Routing:
- net GND: track 22.5 -> 19.3 mm, vias 19 -> 20
Other:
- board size 31.4 x 18.2 mm -> 31.4 x 18.6 mm
Changed lines of the file:
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@@
 		(tags "capacitor handsolder")
 		(property "Reference" "C6"
-			(at 0 -1.43 360)
+			(at 0 -1.43 0)
 			(layer "F.SilkS")
 			(hide yes)
@@
 		)
 		(property "Value" "100n"
-			(at 0 1.43 360)
+			(at 0 1.43 0)
 			(layer "F.Fab")
 			(effects
@@
 		)
 		(fp_text user "${REFERENCE}"
-			(at 0 0 360)
+			(at 0 0 0)
 			(layer "F.Fab")
 			(effects
@@
 		(tags "diode handsolder")
 		(property "Reference" "D1"
-			(at 0 -1.43 360)
+			(at 0 -1.43 0)
 			(layer "F.SilkS")
 			(hide yes)
@@
 		)
 		(property "Value" "1n4148"
-			(at 0 1.43 360)
+			(at 0 1.43 0)
 			(layer "F.Fab")
 			(effects
@@
 		)
 		(fp_text user "${REFERENCE}"
-			(at 0 0 360)
+			(at 0 0 0)
 			(layer "F.Fab")
 			(effects
@@
 		)
 		(fp_text user "${REFERENCE}"
-			(at 0 2.54 360)
+			(at 0 2.54 0)
 			(layer "F.Fab")
 			(effects
@@
 	(footprint "Connector_PinHeader_2.54mm:PinHeader_1x03_P2.54mm_Vertical"
 		(layer "F.Cu")
-		(at 152.5 88.36)
+		(at 152.6032 88.392)
 		(descr "Through hole straight pin header, 1x03, 2.54mm pitch, single row")
 		(tags "Through hole pin header THT 1x03 2.54mm single row")
@@
 		)
 		(fp_text user "${REFERENCE}"
-			(at 0 1.27 360)
+			(at 0 1.27 0)
 			(layer "F.Fab")
 			(effects
@@
 	)
 	(gr_rect
-		(start 124.5 82)
+		(start 124.5 81.5936)
 		(end 155.9 100.2)
 		(stroke
@@
 	)
 	(segment
-		(start 152.5 89.8)
-		(end 152.5 89.85)
-		(width 0)
-		(layer "F.Cu")
-		(net 0)
-	)
-	(segment
 		(start 134.875 96.92)
 		(end 131.755 96.92)
@@
 	)
 	(segment
-		(start 148.9 97.04)
-		(end 152.5 93.44)
+		(start 146.025 85.125)
+		(end 145.049265 84.149265)
 		(width 0.2)
 		(layer "F.Cu")
@@
 	)
 	(segment
-		(start 152.5 93.44)
-		(end 153.475735 94.415735)
+		(start 147.9375 84.3)
+		(end 146.9 84.3)
 		(width 0.2)
 		(layer "F.Cu")
@@
 	)
 	(segment
-		(start 146.025 85.125)
-		(end 145.049265 84.149265)
+		(start 147.075 85.125)
+		(end 146.3 85.125)
 		(width 0.2)
 		(layer "F.Cu")
@@
 	)
 	(segment
-		(start 147.9375 84.3)
-		(end 146.9 84.3)
+		(start 151.5872 93.472)
+		(end 150.7744 92.6592)
 		(width 0.2)
 		(layer "F.Cu")
@@
 	)
 	(segment
-		(start 147.075 85.125)
-		(end 146.3 85.125)
+		(start 147.75 85.8)
+		(end 147.075 85.125)
 		(width 0.2)
 		(layer "F.Cu")
@@
 	)
 	(segment
-		(start 147.75 85.8)
-		(end 147.075 85.125)
+		(start 151.0792 94.996)
+		(end 151.0792 95.1992)
+		(width 0.2)
+		(layer "F.Cu")
+		(net 7)
+	)
+	(segment
+		(start 152.6032 93.472)
+		(end 151.0792 94.996)
 		(width 0.2)
 		(layer "F.Cu")
@@
 	)
 	(segment
-		(start 153.475735 94.415735)
-		(end 153.475735 95.675735)
+		(start 152.6032 93.472)
+		(end 151.5872 93.472)
 		(width 0.2)
 		(layer "F.Cu")
@@
 	)
 	(via
-		(at 147.7 96.2)
+		(at 151.0792 95.1992)
 		(size 0.6)
 		(drill 0.3)
@@
 	)
 	(via
-		(at 129.15 89.65)
+		(at 147.7 96.2)
 		(size 0.6)
 		(drill 0.3)
@@
 	)
 	(via
-		(at 140 97.5)
+		(at 129.15 89.65)
 		(size 0.6)
 		(drill 0.3)
 		(layers "F.Cu" "B.Cu")
-		(free yes)
 		(net 7)
 	)
 	(via
-		(at 137 97.5)
+		(at 140 97.5)
 		(size 0.6)
 		(drill 0.3)
@@
 	)
 	(via
-		(at 153.475735 95.675735)
+		(at 137 97.5)
 		(size 0.6)
 		(drill 0.3)
 		(layers "F.Cu" "B.Cu")
+		(free yes)
 		(net 7)
 	)
@@
 	)
 	(via
+		(at 150.7744 92.6592)
+		(size 0.6)
+		(drill 0.3)
+		(layers "F.Cu" "B.Cu")
+		(net 7)
+	)
+	(via
 		(at 137 95.5)
 		(size 0.6)
@@
 	)
 	(segment
-		(start 152.5 87.45)
-		(end 152.5 88.36)
+		(start 152.6032 88.392)
+		(end 152.6032 87.5532)
 		(width 0.2)
 		(layer "F.Cu")
@@
 	(segment
 		(start 149.6625 84.3)
-		(end 149.6625 83.7625)
+		(end 148.5729 83.2104)
 		(width 0.2)
 		(layer "F.Cu")
@@
 	)
 	(segment
-		(start 149.6625 83.7625)
-		(end 149 83.1)
+		(start 143.7 84.65)
+		(end 143.7 85.9)
 		(width 0.2)
 		(layer "F.Cu")
@@
 	)
 	(segment
-		(start 150.85 85.8)
-		(end 152.5 87.45)
+		(start 146.648529 83.2)
+		(end 145.15 83.2)
 		(width 0.2)
 		(layer "F.Cu")
@@
 	)
 	(segment
-		(start 149 83.1)
-		(end 145.25 83.1)
+		(start 145.15 83.2)
+		(end 143.7 84.65)
 		(width 0.2)
 		(layer "F.Cu")
@@
 	)
 	(segment
-		(start 145.25 83.1)
-		(end 143.7 84.65)
+		(start 146.658929 83.2104)
+		(end 146.648529 83.2)
 		(width 0.2)
 		(layer "F.Cu")
@@
 	)
 	(segment
-		(start 143.7 84.65)
-		(end 143.7 85.9)
+		(start 152.6032 87.5532)
+		(end 150.85 85.8)
 		(width 0.2)
 		(layer "F.Cu")
@@
 	)
 	(segment
-		(start 152.9 97.1)
-		(end 151.44 97.1)
+		(start 148.5729 83.2104)
+		(end 146.658929 83.2104)
+		(width 0.2)
+		(layer "F.Cu")
+		(net 10)
+	)
+	(segment
+		(start 151.44 97.1)
+		(end 152.9 97.1)
 		(width 0.2)
 		(layer "F.Cu")
@@
 	)
 	(segment
-		(start 154.2 91.55)
-		(end 154.2 95.8)
+		(start 153.416 90.932)
+		(end 152.6032 90.932)
 		(width 0.2)
 		(layer "F.Cu")
@@
 	)
 	(segment
-		(start 154.2 95.8)
-		(end 152.9 97.1)
+		(start 154.2 91.716)
+		(end 153.416 90.932)
 		(width 0.2)
 		(layer "F.Cu")
@@
 	)
 	(segment
-		(start 153.55 90.9)
-		(end 154.2 91.55)
+		(start 152.9 97.1)
+		(end 154.2 95.8)
 		(width 0.2)
 		(layer "F.Cu")
@@
 	)
 	(segment
-		(start 152.5 90.9)
-		(end 153.55 90.9)
+		(start 154.2 95.8)
+		(end 154.2 91.716)
 		(width 0.2)
 		(layer "F.Cu")

Commit message: added labeling to the pcb and made gerber 'wq
Other:
- board text added: "*"
- board text added: "+"
- board text added: "-"
- board text added: "G"
- board text added: "In"
- board text added: "O"
- board text added: "Tone"
- board text added: "V"
- board text added: "bat"
- board text added: "out"
Changed lines of the file:
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@@
 			(outputformat 1)
 			(mirror no)
-			(drillshape 1)
+			(drillshape 0)
 			(scaleselection 1)
-			(outputdirectory "")
+			(outputdirectory "manufacturing/")
 		)
 	)
@@
 		)
 	)
+	(gr_circle
+		(center 136.95 89.095576)
+		(end 137.19 89.315576)
+		(stroke
+			(width 0.1)
+			(type default)
+		)
+		(fill none)
+		(layer "F.SilkS")
+	)
 	(gr_rect
 		(start 124.5 81.5936)
@@
 		(layer "Edge.Cuts")
 	)
+	(gr_text "out"
+		(at 148.68 99.77 0)
+		(layer "F.SilkS")
+		(effects
+			(font
+				(size 1 1)
+				(thickness 0.1)
+			)
+			(justify left bottom)
+		)
+	)
+	(gr_text "*"
+		(at 150.26 91.64 0)
+		(layer "F.SilkS")
+		(effects
+			(font
+				(size 1 1)
+				(thickness 0.1)
+			)
+			(justify left bottom)
+		)
+	)
+	(gr_text "+"
+		(at 128.63 88.15 0)
+		(layer "F.SilkS")
+		(effects
+			(font
+				(size 1 1)
+				(thickness 0.1)
+			)
+			(justify left bottom)
+		)
+	)
+	(gr_text "+"
+		(at 132.31 94.47 0)
+		(layer "F.SilkS")
+		(effects
+			(font
+				(size 1 1)
+				(thickness 0.1)
+			)
+			(justify left bottom)
+		)
+	)
+	(gr_text "G"
+		(at 150.23 89.645 0)
+		(layer "F.SilkS")
+		(effects
+			(font
+				(size 1 1)
+				(thickness 0.1)
+			)
+			(justify left bottom)
+		)
+	)
+	(gr_text "In"
+		(at 130.8 86.03 0)
+		(layer "F.SilkS")
+		(effects
+			(font
+				(size 1 1)
+				(thickness 0.1)
+			)
+			(justify left bottom)
+		)
+	)
+	(gr_text "O"
+		(at 154.33 91.45 0)
+		(layer "F.SilkS")
+		(effects
+			(font
+				(size 1 1)
+				(thickness 0.1)
+			)
+			(justify left bottom)
+		)
+	)
+	(gr_text "-\n"
+		(at 154.1 94.04 0)
+		(layer "F.SilkS")
+		(effects
+			(font
+				(size 1 1)
+				(thickness 0.1)
+			)
+			(justify left bottom)
+		)
+	)
+	(gr_text "Tone"
+		(at 139.89 84.57 0)
+		(layer "F.SilkS")
+		(effects
+			(font
+				(size 1 1)
+				(thickness 0.1)
+			)
+			(justify left bottom)
+		)
+	)
+	(gr_text "*"
+		(at 137.81 84.48 0)
+		(layer "F.SilkS")
+		(effects
+			(font
+				(size 1 1)
+				(thickness 0.1)
+			)
+			(justify left bottom)
+		)
+	)
+	(gr_text "*"
+		(at 150.3 88.98 0)
+		(layer "F.SilkS")
+		(effects
+			(font
+				(size 1 1)
+				(thickness 0.1)
+			)
+			(justify left bottom)
+		)
+	)
+	(gr_text "V"
+		(at 152.6032 87.062 0)
+		(layer "F.SilkS")
+		(effects
+			(font
+				(size 1 1)
+				(thickness 0.1)
+			)
+			(justify left bottom)
+		)
+	)
+	(gr_text "bat\n"
+		(at 130.09 99.38 0)
+		(layer "F.SilkS")
+		(effects
+			(font
+				(size 1 1)
+				(thickness 0.1)
+			)
+			(justify left bottom)
+		)
+	)
+	(gr_text "+"
+		(at 153.04 97.78 0)
+		(layer "F.SilkS")
+		(effects
+			(font
+				(size 1 1)
+				(thickness 0.1)
+			)
+			(justify left bottom)
+		)
+	)
+	(gr_text "*"
+		(at 140.75 84.34 0)
+		(layer "F.SilkS")
+		(effects
+			(font
+				(size 1 1)
+				(thickness 0.1)
+			)
+			(justify left bottom)
+		)
+	)
 	(segment
