File: Tuner/Tuner.kicad_sch (KiCad schematic)
At the start: 74 parts, among them J1 Barrel_Jack, J2 Input, J3 Conn_01x04_Pin, J4 SWD, J5 output channel, J6 TIM1 output, Q1 NPN, Q2 NPN, Q3 NPN, Q4 NPN, Q5 NPN, SW1 NRST, SW2 SW_SPDT, U1 NE5532, U2 AMS1117-3.3, U3 STM32F411RETx, Y1 16Mhz

Commit message: removed the LED drivers and finished first layout placement for the PCB
Parts:
- removed D10, D2, D3, D4, D5, D6, D7, D8, D9: LED, LED_SMD:LED_1206_3216Metric_Pad1.42x1.75mm_HandSolder, symbol Device:LED
- removed Q1, Q2, Q3, Q4, Q5: NPN, Package_TO_SOT_SMD:SOT-23, symbol Simulation_SPICE:NPN
- removed R10, R11, R12, R13, R14, R15, R16, R8, R9: 470, Resistor_SMD:R_0603_1608Metric_Pad0.98x0.95mm_HandSolder, symbol Device:R
- removed R17, R18, R19, R20, R21: 6k, Resistor_SMD:R_0603_1608Metric_Pad0.98x0.95mm_HandSolder, symbol Device:R
- removed R22, R23, R24, R25, R26: 0, Resistor_SMD:R_0603_1608Metric_Pad0.98x0.95mm_HandSolder, symbol Device:R
- added C12, C14, C6: 1u, Capacitor_SMD:C_0603_1608Metric_Pad1.08x0.95mm_HandSolder, symbol Device:C
- added C13: 10n, Capacitor_SMD:C_0603_1608Metric_Pad1.08x0.95mm_HandSolder, symbol Device:C
- added r4: 22k, Resistor_SMD:R_0603_1608Metric_Pad0.98x0.95mm_HandSolder, symbol Device:R
- SW2: footprint Button_Switch_THT:SW_E-Switch_EG2219_DPDT_Angled -> Button_Switch_SMD:SW_SPDT_PCM12
- renumbered C9 to C10, C10 to C11, C11 to C15, C12 to C16, C6 to C7, C7 to C8, C8 to C9, R27 to R28, R28 to R29, R29 to R30, R30 to R31, R31 to R32, R4 to R5, R5 to R6, R6 to R7, R7 to R8
Connections:
- net +9V: now also C6.1
- net ADC1_IN0: now also C12.2; no longer RV1.1, RV1.2, U1.1
- net GND: now also J2.1 (Pin_1), C13.2, C6.2; no longer J2.2 (Pin_2), R6.1
- net voltage bias: now also R6.1, C14.2
- net at U1.3 (+): now also r4.2; no longer J2.1 (Pin_1)
- net LED_GREEN: no longer names the net of U3.38 (PC7)
- net LED_RED_1: no longer names the net of U3.40 (PC9)
- net LED_RED_2: no longer names the net of U3.52 (PC11)
- net LED_YELLOW_1: no longer names the net of U3.39 (PC8)
- net LED_YELLOW_2: no longer names the net of U3.51 (PC10)
- new net: C12.1, RV1.1, RV1.2, U1.1
- new net: C14.1, J2.2 (Pin_2)
- new net: C13.1, r4.1
- no-connect marks 36 -> 41
Other:
- note removed: "LED driver"
- moved on the sheet: J2, R3, R5, R6, R7, RV1, U1A
